File: 01_Hardware/KiCad/Plantomatic2000.kicad_sch (KiCad schematic)
At the start: 60 parts, among them J201 USB_C_Receptacle_USB2.0_16P, J3 Conn_02x05_Odd_Even, J4 Conn_02x03_Odd_Even, Q1 RS9N50D, Q2 RS9N50D, SW1 SW_Push, SW2 SW_Push, SW202 KSR222G LFS, U1 ESP32-WROOM-32E, U101 XC6220B331MR, U2 nPM1300, U201 USBLC6-2P6, U202 CP2102N-A02-GQFN24

Commit message: Test commit
Parts:
- added J1: Conn_02x05_Odd_Even, symbol Connector_Generic:Conn_02x05_Odd_Even
Changed lines of the file:
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@@
+	)
+	(symbol
+		(lib_id "Connector_Generic:Conn_02x05_Odd_Even")
+		(at 255.27 217.17 0)
+		(unit 1)
+		(exclude_from_sim no)
+		(in_bom yes)
+		(on_board yes)
+		(dnp no)
+		(fields_autoplaced yes)
+		(property "Reference" "J1"
+			(at 256.54 205.74 0)
+			(effects
+				(font
+					(size 1.27 1.27)
+				)
+			)
+		)
+		(property "Value" "Conn_02x05_Odd_Even"
+			(at 256.54 208.28 0)
+			(effects
+				(font
+					(size 1.27 1.27)
+				)
+			)
+		)
+		(property "Footprint" ""
+			(at 255.27 217.17 0)
+			(effects
+				(font
+					(size 1.27 1.27)
+				)
+				(hide yes)
+			)
+		)
+		(property "Datasheet" "~"
+			(at 255.27 217.17 0)
+			(effects
+				(font
+					(size 1.27 1.27)
+				)
+				(hide yes)
+			)
+		)
+		(property "Description" "Generic connector, double row, 02x05, odd/even pin numbering scheme (row 1 odd numbers, row 2 even numbers), script generated (kicad-library-utils/schlib/autogen/connector/)"
+			(at 255.27 217.17 0)
+			(effects
+				(font
+					(size 1.27 1.27)
+				)
+				(hide yes)
+			)
+		)
+		(pin "2"
+		)
+		(pin "6"
+		)
+		(pin "1"
+		)
+		(pin "3"
+		)
+		(pin "5"
+		)
+		(pin "7"
+		)
+		(pin "9"
+		)
+		(pin "4"
+		)
+		(pin "10"
+		)
+		(pin "8"
+		)
+		(instances
+			(project ""
+				(path "/7b3f5236-3811-4a22-865a-1f6a26bdd727"
+					(reference "J1")
+					(unit 1)
+				)
+			)
+		)
 	)
 	(symbol

Commit message: Schematic: Added TPS61287 +12V Boost converter, Datasheet: TPS61287 and preliminary BOM
Parts:
- added C114, C133: 1uF, symbol Device:C_Small
- added C119, C122, C124: 100nF, symbol Device:C_Small
- added C120, C121: 47uF, symbol Device:C_Small
- added C123: 10uF, symbol Device:C_Small
- added C125: 58pF, symbol Device:C_Small
- added C126: 4.7nF, symbol Device:C_Small
- added C127: 2.2uF, symbol Device:C_Small
- added L103: 4.7uH (MLC1565-472MLC), symbol Device:L
- added Q103: CSD17571 N-Channel, symbol Global_Custom_Libb:CSD17571
- added R108: 158K, symbol Device:R
- added R109: 14K3, symbol Device:R
- added R110: 10K, symbol Device:R
- added R111: 20K, symbol Device:R
- added U104: TPS61287, symbol Global_Custom_Libb:TPS61287
- renumbered C206 to C102, C207 to C103, C1 to C104, C2 to C105, C102 to C106, C103 to C107, C104 to C108, C105 to C109, C106 to C110, C3 to C111, C107 to C112, C112 to C113, C7 to C115, C6 to C116, C5 to C117, C4 to C118, C201 to C128, C202 to C129, C203 to C130, C204 to C131, C205 to C132, D103 to D101, D2 to D102, D202 to D103, D203 to D104, D3 to D105, FB201 to FB101, J3 to J101, J4 to J102, J201 to J103, J1 to J104, L1 to L101, L2 to L102, Q1 to Q101, Q2 to Q102, R2 to R101, R1 to R102, R3 to R103, R207 to R104, R5 to R105, R4 to R106, R209 to R107, R201 to R112, R202 to R113, R203 to R114, R204 to R115, R205 to R116, R206 to R117, R208 to R118, R210 to R119, R211 to R120, SW202 to SW101, SW2 to SW102, SW1 to SW103, TP103 to TP101, U2 to U102, U1 to U103, U201 to U105, U202 to U106
Connections:
- net +12V: now also C114.1, C119.1, C120.1, C121.1, C133.1, R108.1, U104.5 (VOUT)
- net +VSYS: now also C123.1, C124.1, L103.1, U104.12 (VIN), U104.13 (EN/UVLO)
- net GND: now also C119.2, C120.2, C121.2, C123.2, C124.2, C125.2, C126.2, C127.2, Q103.4 (Source), Q103.8 (Source), R109.2, R111.1, U104.10 (M/SYNC), U104.14 (AGND), U104.8 (PGND)
- net at L102.2, Q102.2 (D): now also C114.2
- net at L101.2, Q101.2 (D): now also C133.2
- new net: C125.1, R110.1, U104.3 (COMP)
- new net: C126.1, R110.2
- new net: C127.1, U104.11 (VCC), U104.4 (MODE)
- new net: C122.1, L103.2, Q103.1 (Drain), Q103.2 (Drain), Q103.5 (Drain), Q103.6 (Drain), Q103.7 (Drain), U104.6 (SW)
- new net: R108.2, R109.1, U104.2 (FB)
- new net: R111.2, U104.1 (ILIM)
- new net: C122.2, U104.7 (BOOT)
- new net: Q103.3 (Gate), U104.9 (DRV)
Other:
- note added: "+3V4/+5V to +12V Boost Converter"
- note removed: "+5V to +12V Boost Converter"
- note removed: "DRV8212 Brushed motor driver IC"
- note removed: "MPQ3425 BOOST CONVERTER up to 3.5A Current controlled for inductive loads"
- moved on the sheet: J104, L101, L102, Q101, Q102, R102, R103, R105, R106

Commit message: Added DS3231 RTC + datasheets with interuppt wake up from RTC to nPM1300 PMIC
Parts:
- added BT101: Battery_Cell, Battery:BatteryHolder_MYOUNG_BS-07-A1BJ001_CR2032, symbol Device:Battery_Cell
- added C134: 22uF, symbol Device:C_Polarized_Small_US
- added C135: 4.7nF, symbol Device:C_Small
- added C136: 100nF, Capacitor_SMD:C_0402_1005Metric, symbol Device:C_Small
- added C137: 10uF, Capacitor_SMD:C_0402_1005Metric, symbol Device:C_Small
- added D106: 1N4148W, Diode_SMD:D_SOD-123, symbol Diode:1N4148W
- added D107: LED, symbol Device:LED
- added Q104: RS9N50D, Package_TO_SOT_SMD:TO-252-2, symbol Transistor_FET:RS9N50D
- added R121, R124: 10K, symbol Device:R
- added R122: 220R, symbol Device:R
- added R123: 1K, symbol Device:R
- added R125: 470R, symbol Device:R
- added U107: DS3231M, Package_SO:SOIC-16W_7.5x10.3mm_P1.27mm, symbol Timer_RTC:DS3231M
- R111: value 20K -> 40K
Connections:
- net +3V3: now also C136.1, C137.1, R122.2, R123.2, U107.2 (VCC)
- net +VSYS: now also C134.1
- net GND: now also BT101.2 (-), C134.2, C135.2, C136.2, C137.2, D107.1 (K), Q104.3 (S), R124.1, U107.10 (GND), U107.11 (GND), U107.12 (GND), U107.13 (GND), U107.4 (~{RST}), U107.5 (GND), U107.6 (GND), U107.7 (GND), U107.8 (GND), U107.9 (GND)
- net SCL: now also U102.14 (SCL), U107.16 (SCL); no longer U102.13 (SDA)
- net SDA: now also U102.13 (SDA), U107.15 (SDA); no longer U102.14 (SCL)
- net SHPHLD: now also U103.26 (IO4), Q104.2 (D)
- net at C122.1, L103.2, Q103.1 (Drain)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: now also R121.1
- new net: D106.2 (A), R122.1
- new net: C135.1, R121.2
- new net: BT101.1 (+), D106.1 (K), U107.14 (VBAT)
- new net: D107.2 (A), R123.1
- new net: Q104.1 (G), R125.2
- new net: R124.2, R125.1, U107.3 (~{INT}/SQW)
Other:
- note added: "ESP32 WROOM 32E"
- note added: "IL peak = Idc+(Ipp/2) IL peak = 7.84A+(1.65A/2) = 8.66A Inductor must have a higher saturation current of 9A"
- note added: "Peak to Peak Inductor Current Ripple Ipp = 1/L*[(1/(Vout-Vin))+(1/Vin)]*fsw OR Ipp = (Vin*D)/(L*fsw) Ipp = (3.4V * 0.73%) / (4.7uH*340KHz) = 1.65A"
- note added: "RTC DS3231"
- note added: "Rlim = 400K / A Rlin = 400K / 10A = 40K"
- note added: "VOUT = 12V VREF = 1V R109 = 14K3 R108 = [(VOUT - VREF) * R109]/VREF R108 = [(12 - 1)* 14300]/1 = 157300 or 158K R108 = 158K"
- note added: "Vripple_dis = [(VOUT-VIN)*IOUT]/VOUT*fsw*Cout Vripple_dis = [12V-3.4V*2A]/12*320KHz*(47uF*2) = 48mV Vripp_ESR = ILpeak*Rc_esr Vripp_ESR = 8.66A*30mOhms (at 320KHz esr between 10-50mOhms) = 260mV"
- note added: "n = power convertion efficiency Idc = (VOUT*IOUT)/(VIN*n) Idc = (12V*2A)/(3.4V*90%) = 7.84A"
- moved on the sheet: C119, C120, C121, C122, C123, C124, C125, C126, C127, J104, L103, Q103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

Commit message: Schematic: Added enable circuitry for Display, Water Sensor and Boost converter. Also connectors, LED's, EEPROM, USB to Serial Programming (RTS and DTR). Added datasheets and simulation of Enable circuitry
Parts:
- removed D101: LED_ARGB, LED_SMD:LED_Wurth_150044M155260, symbol Device:LED_ARGB
- removed J104: Conn_02x05_Odd_Even, symbol Connector_Generic:Conn_02x05_Odd_Even
- removed L101: Pump_1, symbol Device:L
- removed L102: Pump_2, symbol Device:L
- removed SW101: KSR222G LFS, Button_Switch_SMD:SW_Tactile_SPST_NO_Straight_CK_PTS636Sx25SMTRLFS, symbol Switch:SW_Push
- added C138, C139, C140, C141, C142, C143, C146, C147, C148: 100nF, symbol Device:C_Small
- added C144: 10uF, Capacitor_SMD:C_0402_1005Metric, symbol Device:C_Small
- added C145: 100nF, Capacitor_SMD:C_0402_1005Metric, symbol Device:C_Small
- added D108, D109: D, symbol Device:D
- added J104: PMIC RGB LED, symbol Connector_Generic:Conn_01x04
- added J105: OLED Display, symbol Connector_Generic:Conn_01x04
- added J106: Line Select, symbol Connector_Generic:Conn_01x02
- added J107: Manual Start, symbol Connector_Generic:Conn_01x02
- added J108: Hour, symbol Connector_Generic:Conn_01x02
- added J109: Minute, symbol Connector_Generic:Conn_01x02
- added J110: Water Sensor, symbol Connector_Generic:Conn_01x04
- added J111: System Reset, symbol Connector_Generic:Conn_01x02
- added J112, J113: Conn_01x02, symbol Connector_Generic:Conn_01x02
- added J114: System Wake Up, symbol Connector_Generic:Conn_01x02
- added J115: Running LED, symbol Connector_Generic:Conn_01x02
- added JP101: ModSel, symbol Jumper:SolderJumper_3_Open
- added Q105, Q108, Q110: PMOS, symbol Simulation_SPICE:PMOS
- added Q106, Q107, Q109: RS9N50D, Package_TO_SOT_SMD:TO-252-2, symbol Transistor_FET:RS9N50D
- added Q111, Q112: DTC143Z, Package_TO_SOT_SMD:SOT-23-3, symbol Transistor_BJT:DTC143Z
- added R126, R129, R130, R132, R140, R142: 10K, symbol Device:R
- added R127, R128, R131, R133, R139, R141, R143: 470R, symbol Device:R
- added R134, R135, R136, R137, R138, R147: 0R, symbol Device:R
- added R144, R145, R151, R152, R153: 4K7, Resistor_SMD:R_0402_1005Metric, symbol Device:R
- added R146: 0R, Resistor_SMD:R_0402_1005Metric, symbol Device:R
- added R148, R149, R150: 220R, Resistor_SMD:R_0402_1005Metric, symbol Device:R
- added R155, R157, R158: 12K, symbol Device:R
- added R156: 470R, Resistor_SMD:R_0402_1005Metric, symbol Device:R
- added R159: 5K1, symbol Device:R
- added U108: AT24CS01-SSHM, Package_SO:SOIC-8_3.9x4.9mm_P1.27mm, symbol Memory_EEPROM:AT24CS01-SSHM
- C135, R121: now not fitted
- R107, R114, R115: value 0R -> 470R
- R123: value 1K -> 470R
Connections:
- net +12V: now also D108.1 (K), D109.1 (K), J112.1 (Pin_1), J113.1 (Pin_1), Q110.3 (S), R142.2
- net +3V3: now also R104.2, C144.1, C145.1, C147.1, Q105.3 (S), R129.2, R139.2, R144.1, R145.1, R151.1, R152.1, R153.1, U108.8 (VCC); no longer R104.1
- net +VSYS: now also C148.1, J104.4 (Pin_4), Q108.3 (S), R132.2; no longer U104.13 (EN/UVLO)
- net ESP_EN: now also Q111.3 (C), R158.1
- net ESP_IO0: now also Q112.3 (C), R156.1, R159.1; no longer C117.1, SW102.2
- net GND: now also U106.23 (~{DTR}), C138.2, C139.2, C140.2, C141.2, C142.2, C143.2, C144.2, C145.2, C146.2, C147.2, C148.2, J105.4 (Pin_4), J106.2 (Pin_2), J107.2 (Pin_2), J108.2 (Pin_2), J109.2 (Pin_2), J110.4 (Pin_4), J111.2 (Pin_2), J114.2 (Pin_2), J115.2 (Pin_2), JP101.3 (B), Q106.3 (S), Q107.3 (S), Q109.3 (S), Q112.2 (E), R126.1, R130.1, R140.1, R157.1, U108.4 (GND), U108.7 (WP)
- net SCL: now also J105.2 (Pin_2), R144.2, R146.2, U108.6 (SCL)
- net SDA: now also U103.36 (IO22), J105.1 (Pin_1), R145.2, U108.5 (SDA)
- net VBUS: now also C115.1, C116.1, J101.1 (Pin_1), J102.2 (Pin_2)
- net VBUSD: no longer C115.1, C116.1, J101.1 (Pin_1), J102.2 (Pin_2)
- net VDD: now also C146.1, R158.2, R159.2
- net at C127.1, U104.11 (VCC): now also JP101.1 (A); no longer U104.4 (MODE)
- net at C114.2, Q102.2 (D): now also D109.2 (A), J112.2 (Pin_2)
- net at U102.25 (LED0): now also R148.2
- net at U102.26 (LED1): now also R149.2
- net at U102.27 (LED2): now also R150.2
- net at U103.27 (IO16): now also R104.1; no longer R104.2
- net RTS_SERIAL: now reaches U106.19 (~{RTS})
- net RTS_SERIAL: now also Q111.2 (E), R155.1
- net at C133.2, Q101.2 (D): now also D108.2 (A), J113.2 (Pin_2)
- net SELECT_LINE_BUTTON_PIN: now reaches U103.10 (IO25)
- net SELECT_LINE_BUTTON_PIN: now also R135.2
- net MIN_BUTTON_PIN: now reaches U103.11 (IO26)
- net MIN_BUTTON_PIN: now also R138.2
- net HOUR_BUTTON_PIN: now reaches U103.12 (IO27)
- net HOUR_BUTTON_PIN: now also R137.2
- net DISPLAY_EN: now reaches U103.24 (IO2)
- net PUMP2_EN: now reaches U103.30 (IO18)
- net PUMP2_EN: now also R105.1, R106.2
- net PUMP1_EN: now reaches U103.31 (IO19)
- net PUMP1_EN: now also R102.1, R103.2
- net at U103.33 (IO21): now also R146.1
- net WATER_SENSOR_EN: now reaches U103.37 (IO23)
- net WATER_SENSOR_EN: now also R140.2, R141.1
- net BOOST_ENABLE: now reaches U103.6 (IO34)
- net BOOST_ENABLE: now also R130.2, R131.1
- net DISPLAY_ENABLE: now reaches U103.7 (IO35)
- net DISPLAY_ENABLE: now also R126.2, R127.1
- net PMIC_SHPHLD: now reaches U103.8 (IO32)
- net PMIC_SHPHLD: now also Q104.2 (D), U102.15 (SHPHLD), R134.2
- net RESET_BUTTON_PIN: now reaches U103.9 (IO33)
- net RESET_BUTTON_PIN: now also R147.2
- net ESP_TMS renamed START_BUTTON_PIN
- net START_BUTTON_PIN: now also R136.2
- removed net Pump_Drive_1: R102.1, R103.2, R105.1, R106.2
- removed net SHPHLD: Q104.2 (D), U102.15 (SHPHLD), U103.26 (IO4)
- new net: C143.1, J111.1 (Pin_1), R147.1
- new net: J115.1 (Pin_1), R139.1
- new net: J110.3 (Pin_3), Q110.1 (D)
- new net: Q110.2 (G), R142.1, R143.2
- new net: C139.1, J106.1 (Pin_1), R135.1
- new net: Q105.2 (G), R128.2, R129.1
- new net: Q106.1 (G), R127.2
- new net: Q106.2 (D), R128.1
- new net: Q109.1 (G), R141.2
- new net: J105.3 (Pin_3), Q105.1 (D)
- new net: C138.1, J114.1 (Pin_1), R134.1
- new net: R151.2, U108.1 (A0)
- new net: Q108.1 (D), U104.13 (EN/UVLO)
- new net: JP101.2 (C), U104.4 (MODE)
- new net: C141.1, J108.1 (Pin_1), R137.1
- new net: Q109.2 (D), R143.1
- new net: Q112.1 (B), R155.2
- new net: Q107.1 (G), R131.2
- new net: Q107.2 (D), R133.1
- new net: Q108.2 (G), R132.1, R133.2
- new net: C142.1, J109.1 (Pin_1), R138.1
- new net: C140.1, J107.1 (Pin_1), R136.1
- new net: J104.2 (Pin_2), R149.1
- new net: J104.3 (Pin_3), R148.1
- new net: C117.1, R156.2, SW102.2
- new net: R153.2, U108.3 (A2)
- new net: Q111.1 (B), R157.2
- new net: R152.2, U108.2 (A1)
- new net: J104.1 (Pin_1), R150.1
- new net WATER_SENSOR_SIG: U103.26 (IO4)
- no-connect marks 38 -> 23
Other:
- note added: "EEPROM"
- note added: "Hour"
- note added: "Line Select"
- note added: "Manual Start"
- note added: "Minute"
- note added: "OLED Display"
- note added: "Running LED"
- note added: "System Reset"
- note added: "System WakeUp"
- note added: "TO DO: CHECK MOSFET PINOUT IF GATE / DRAIN / SOURCE ARE CORRECT FIND CONNECTORS AND CHECK FOOTPRINT CHECK CONNECTOR ORIENTATION FOR RESET / PUMP1 / PUMP2 / DISPLAY / WATER SENSOR / RUNNING LED / RGB LED ANOTATE SCHEMATIC CREATE FOOTPRINTS ASSIGN FOOTPRINTS MAKE BOM DESIGN PCB"
- note added: "USB to SERIAL PROGRAMMING"
- note added: "User Interface Buttons"
- note added: "VDD is supplied by the VDD pin of CP2102N When USB C is removed the CP2102N should power OFF"
- note added: "Water Sensor"
- note removed: "TO DO: New BOOST converter that can handle up to 3A Find a replacement for the HEXFET (IGBT) on the optocoupler input Find the connector for the pumps"
- moved on the sheet: BT101, C114, C115, C116, C117, C118, C119, C120, C121, C122, C123, C124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

Commit message: Added foorptrints
Parts:
- removed J104: PMIC RGB LED, symbol Connector_Generic:Conn_01x04
- removed Q103: CSD17571 N-Channel, symbol Global_Custom_Libb:CSD17571
- removed R101: 10K, symbol Device:R_US
- added J116: JST_4B4, Connector_JST:JST_EH_B4B-EH-A_1x04_P2.50mm_Vertical, symbol Connector_Generic:Conn_01x04
- added Q113: CSD17313Q2, Package_SON:Texas_DQK, symbol Transistor_FET:CSD17313Q2
- added R154: 10K, Resistor_SMD:R_0402_1005Metric, symbol Device:R
- C103, C107, C108, C109, C110: footprint Capacitor_SMD:C_0402_1005Metric -> Capacitor_SMD:C_0603_1608Metric
- C104, C114, C120, C121, C123, C127, C133, C134: footprint (none) -> Capacitor_SMD:C_0603_1608Metric
- C105, C111, C115, C116, C117, C118, C119, C122, C124, C125, C126, C135, C138, C139, C140, C141, C142, C143, C146, C147, C148: footprint (none) -> Capacitor_SMD:C_0402_1005Metric
- D108, D109: value D -> SS14; footprint (none) -> Custom_Global_Footprints:SS14
- J105: value OLED Display -> JST_B4B; footprint (none) -> Connector_JST:JST_EH_B4B-EH-A_1x04_P2.50mm_Vertical
- J106, J107, J108, J109, J111, J114, J115: footprint (none) -> Connector_JST:JST_EH_B2B-EH-A_1x02_P2.50mm_Vertical
- J110: value Water Sensor -> JST_4B4; footprint (none) -> Connector_JST:JST_EH_B4B-EH-A_1x04_P2.50mm_Vertical
- J112, J113: value Conn_01x02 -> JST_B2B; footprint (none) -> Connector_JST:JST_EH_B2B-EH-A_1x02_P2.50mm_Vertical
- Q101, Q102: value RS9N50D -> IRLL014NTRPBF; footprint Package_TO_SOT_SMD:TO-252-2 -> Package_TO_SOT_SMD:SOT-223
- Q104, Q106, Q107, Q109: value RS9N50D -> NVTA7002NT1G; footprint Package_TO_SOT_SMD:TO-252-2 -> Package_TO_SOT_SMD:SOT-323_SC-70
- Q105, Q108, Q110: value PMOS -> RU1E002SPTCL; footprint (none) -> Package_TO_SOT_SMD:SOT-323_SC-70
- R102, R103, R105, R106, R108, R109, R110, R111, R121, R122, R123, R124, R125, R126, R127, R128, R129, R130, R131, R132, R134, R135, R136, R137, R138, R139, R140, R141, R142, R143, R147, R155, R157, R158, R159: footprint (none) -> Resistor_SMD:R_0402_1005Metric
- R133: value 470R -> 10K; footprint (none) -> Resistor_SMD:R_0402_1005Metric
Connections:
- net DISPLAY_EN is gone; now on net DISPLAY_ENABLE: U103.24 (IO2)
- net +12V: now also J112.2 (Pin_2), J113.2 (Pin_2); no longer J112.1 (Pin_1), J113.1 (Pin_1)
- net +3V3: now also R154.1
- net +VSYS: now also J116.4 (Pin_4)
- net DISPLAY_ENABLE: no longer U103.7 (IO35)
- net ESP_EN: now also R154.2
- net GND: now also J105.1 (Pin_1), J106.1 (Pin_1), J107.1 (Pin_1), J108.1 (Pin_1), J109.1 (Pin_1), J110.3 (Pin_3), J111.1 (Pin_1), J114.1 (Pin_1), J115.1 (Pin_1), Q113.4 (S), Q113.7 (S); no longer J105.4 (Pin_4), J106.2 (Pin_2), J107.2 (Pin_2), J108.2 (Pin_2), J109.2 (Pin_2), J111.2 (Pin_2), J114.2 (Pin_2), J115.2 (Pin_2)
- net SCL: now also J105.3 (Pin_3); no longer J105.2 (Pin_2)
- net SDA: now also J105.4 (Pin_4); no longer J105.1 (Pin_1)
- net WATER_SENSOR_SIG: now also J110.2 (Pin_2)
- net at C143.1, R147.1: now also J111.2 (Pin_2); no longer J111.1 (Pin_1)
- net at R139.1: now also J115.2 (Pin_2); no longer J115.1 (Pin_1)
- net at Q110.1 (D): now also J110.1 (Pin_1); no longer J110.3 (Pin_3)
- net at C114.2, D109.2 (A), Q102.2 (D): now also J112.1 (Pin_1); no longer J112.2 (Pin_2)
- net at C139.1, R135.1: now also J106.2 (Pin_2); no longer J106.1 (Pin_1)
- net at C122.1, L103.2, R121.1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: now also Q113.1 (D), Q113.2 (D), Q113.5 (D), Q113.6 (D), Q113.8 (D)
- net at Q105.1 (D): now also J105.2 (Pin_2); no longer J105.3 (Pin_3)
- net at C138.1, R134.1: now also J114.2 (Pin_2); no longer J114.1 (Pin_1)
- net at U104.9 (DRV): now also Q113.3 (G)
- net at C133.2, D108.2 (A), Q101.2 (D): now also J113.1 (Pin_1); no longer J113.2 (Pin_2)
- net at C141.1, R137.1: now also J108.2 (Pin_2); no longer J108.1 (Pin_1)
- net at C142.1, R138.1: now also J109.2 (Pin_2); no longer J109.1 (Pin_1)
- net at C140.1, R136.1: now also J107.2 (Pin_2); no longer J107.1 (Pin_1)
- net at R149.1: now also J116.2 (Pin_2)
- net at R148.1: now also J116.3 (Pin_3)
- net at R150.1: now also J116.1 (Pin_1)
Other:
- note added: "ADD Linear Regulator for Water Sensor to filter noise"
- note added: "ESP32: GPIO4 INTERNAL PULL UP TO 3V3 WATER SENSOR: GPIO4 to PIN2 (THE WATER SENSOR SIGNAL)"
- moved on the sheet: J110, J112, J113, J115, Q109, Q110, R140, R141, R142, R143

Commit message: Finised assigning footprints
Parts:
- removed D102: BAT760-7, symbol Device:D
- removed D105: UCLAMP6061P.TNT, Diode_SMD:D_MiniMELF, symbol Diode:BZV55B3V9
- removed Q101, Q102: IRLL014NTRPBF, Package_TO_SOT_SMD:SOT-223, symbol Transistor_FET:RS9N50D
- added D110: SS14, Custom_Global_Footprints:SS14M_Flyback_Diode, symbol Device:D
- added D111, D112, D113, D114: SML-P12U2TT86R, LED_SMD:LED_0402_1005Metric, symbol Device:LED
- added Q101, Q102: IRLL014NP, Package_TO_SOT_SMD:SOT-223, symbol Global_Custom_Libb:IRLL014N_HEXFET
- added R160, R161, R162, R163: 1K, Resistor_SMD:R_0402_1005Metric, symbol Device:R
- D103, D104: value LTST-C193KGKT-5A -> SML-P13PTT86R; footprint Custom_Global_Footprints:LTST-C193KGKT-5A -> LED_SMD:LED_0402_1005Metric
- D107: value LED -> SML-P12U2TT86R; footprint (none) -> LED_SMD:LED_0402_1005Metric
- D108, D109: footprint Custom_Global_Footprints:SS14 -> Custom_Global_Footprints:SS14M_Flyback_Diode
- J101: footprint (none) -> Connector_PinHeader_1.27mm:PinHeader_2x05_P1.27mm_Vertical_SMD
- J102: footprint (none) -> Connector_PinHeader_1.27mm:PinHeader_2x03_P1.27mm_Vertical_SMD
- JP101: footprint (none) -> Jumper:SolderJumper-3_P1.3mm_Open_RoundedPad1.0x1.5mm
- L103: value 4.7uH (MLC1565-472MLC) -> 4.7uH (SPM12565VT-4R7M-D); footprint (none) -> Custom_Global_Footprints:SPM12565VT-4R7M
- R123: value 470R -> 1K
- R128, R143: value 470R -> 10K
- SW102, SW103: footprint (none) -> Button_Switch_SMD:SW_SPST_PTS645
- U104: footprint (none) -> Custom_Global_Footprints:RZP0014A-MFG
Connections:
- net GND: now also D111.1 (K), D112.1 (K), D113.1 (K), D114.1 (K), Q101.3 (S), Q102.3 (S)
- net VBUS: now also D110.1 (K)
- net VBUSD: now also D110.2 (A)
- net VDD: now also R163.2
- net at J110.1 (Pin_1), Q110.1 (D): now also R161.2
- net at C114.2, D109.2 (A), J112.1 (Pin_1): now also Q102.2 (D), Q102.4 (D)
- net at J105.2 (Pin_2), Q105.1 (D): now also R162.2
- net at Q108.1 (D), U104.13 (EN/UVLO): now also R160.2
- net at C133.2, D108.2 (A), J113.1 (Pin_1): now also Q101.2 (D), Q101.4 (D)
- net at R105.2: now also Q102.1 (G)
- net at R102.2: now also Q101.1 (G)
- new net: D114.2 (A), R163.1
- new net: D112.2 (A), R161.1
- new net: D111.2 (A), R160.1
- new net: D113.2 (A), R162.1
Other:
- moved on the sheet: C114, C133, D107, D108, D109, J112, J113, Q105, Q106, Q107, Q108, R123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

Commit message: Added test points and schematic.pdf file
Parts:
- added TP102, TP103, TP104, TP105, TP106, TP107, TP108, TP109, TP110, TP111, TP112, TP113, TP114, TP115, TP116, TP117, TP118, TP119, TP120, TP121, TP122, TP123, TP124, TP125, TP126, TP127, TP128, TP129, TP130, TP131, TP132, TP133, TP134, TP135, TP136, TP137: ~, TestPoint:TestPoint_Pad_D1.0mm, symbol Connector:TestPoint
- R139: value 470R -> 1K
- R148, R149, R150: value 220R -> 1K
Connections:
- net +12V: now also TP125.1
- net +3V3: now also TP103.1
- net +VSYS: now also TP102.1, TP121.1
- net ESP_EN: now also TP130.1
- net ESP_RX: now also TP128.1
- net ESP_TX: now also TP129.1
- net PMIC_SHPHLD: now also TP120.1
- net SCL: now also TP117.1
- net SDA: now also TP118.1
- net VBUS: now also TP115.1, TP119.1
- net VDD: now also TP116.1
- net at C143.1, J111.2 (Pin_2), R147.1: now also TP136.1
- net at J110.1 (Pin_1), Q110.1 (D), R161.2: now also TP109.1
- net at Q110.2 (G), R142.1, R143.2: now also TP111.1
- net at C114.2, D109.2 (A), J112.1 (Pin_1)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: now also TP105.1
- net at C139.1, J106.2 (Pin_2), R135.1: now also TP132.1
- net at Q105.2 (G), R128.2, R129.1: now also TP113.1
- net at Q106.1 (G), R127.2: now also TP112.1
- net at Q109.1 (G), R141.2: now also TP110.1
- net at C122.1, L103.2, Q113.1 (D)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: now also TP122.1
- net at J105.2 (Pin_2), Q105.1 (D), R162.2: now also TP114.1
- net at R108.2, R109.1, U104.2 (FB): now also TP124.1
- net at C138.1, J114.2 (Pin_2), R134.1: now also TP131.1
- net at Q108.1 (D), R160.2, U104.13 (EN/UVLO): now also TP137.1
- net at Q113.3 (G), U104.9 (DRV): now also TP123.1
- net at C133.2, D108.2 (A), J113.1 (Pin_1)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: now also TP104.1
- net at C141.1, J108.2 (Pin_2), R137.1: now also TP134.1
- net at Q107.1 (G), R131.2: now also TP127.1
- net at Q108.2 (G), R132.1, R133.2: now also TP126.1
- net at C142.1, J109.2 (Pin_2), R138.1: now also TP135.1
- net at Q101.1 (G), R102.2: now also TP107.1
- net at C140.1, J107.2 (Pin_2), R136.1: now also TP133.1
- net at Q102.1 (G), R105.2: now also TP106.1
- net at Q104.1 (G), R125.2: now also TP108.1
Other:
- note added: "TO DO: BOM DESIGN PCB"
- note removed: "TO DO: CHECK MOSFET PINOUT IF GATE / DRAIN / SOURCE ARE CORRECT FIND CONNECTORS AND CHECK FOOTPRINT CHECK CONNECTOR ORIENTATION FOR RESET / PUMP1 / PUMP2 / DISPLAY / WATER SENSOR / RUNNING LED / RGB LED ANOTATE SCHEMATIC CREATE FOOTPRINTS ASSIGN FOOTPRINTS MAKE BOM DESIGN PCB"
- moved on the sheet: D112, D113, R126, R127, R130, R131, R140, R141, R161, R162

Commit message: PCB layout BOOST converter
Parts:
- removed FB101: MH2029-300Y, Resistor_SMD:R_0805_2012Metric, symbol Device:FerriteBead
- added J117: Running LED, Connector_JST:JST_EH_B2B-EH-A_1x02_P2.50mm_Vertical, symbol Connector_Generic:Conn_01x02
- added R164: 0R, Resistor_SMD:R_0402_1005Metric, symbol Device:R
- C102: value 100nF -> 100nF tantulum; footprint Capacitor_SMD:C_0402_1005Metric -> Capacitor_SMD:C_1206_3216Metric
- C103: value 10uF -> 10uF tantulum; footprint Capacitor_SMD:C_0603_1608Metric -> Capacitor_SMD:C_1206_3216Metric
- C107, C108: footprint Capacitor_SMD:C_0603_1608Metric -> Capacitor_SMD:C_0402_1005Metric
- R114, R115: value 470R -> 0R
Connections:
- net +VBAT: now also J117.2 (Pin_2)
- net +VSYS: now also L103.2; no longer L103.1
- net ESP_TX: now also R164.2; no longer U103.35 (TXD0/IO1)
- net GND: now also J117.1 (Pin_1); no longer Q112.2 (E), R157.1, U106.23 (~{DTR})
- net CVCC: now reaches C127.1, JP101.1 (A), U104.11 (VCC)
- net SW: now reaches C122.1, Q113.1 (D), Q113.2 (D), Q113.5 (D), Q113.6 (D), Q113.8 (D), R121.1, TP122.1, U104.6 (SW)
- net SW: now also L103.1; no longer L103.2
- net SHIELD: no longer names the net of J103.S1 (SHIELD)
- new net: R164.1, U103.35 (TXD0/IO1)
- new net DTR_SERIAL: Q112.2 (E), R157.1, U106.23 (~{DTR})
- no-connect marks 23 -> 25
Other:
- moved on the sheet: C103, C112, L103, TP129
