File: 01_Hardware/KiCad_v2/Plantomatic2000.kicad_sch (KiCad schematic)
At the start: 202 parts, among them J101 Conn_02x05_Odd_Even, J102 Conn_02x03_Odd_Even, J103 USB_C_Receptacle_USB2.0_16P, J105 JST_B4B, J106 JST_B2B, J107 JST_B2B, J108 JST_B2B, J109 JST_B2B, J110 JST_B4B, J111 JST_B2B, J112 JST_B2B, J113 JST_B2B, J114 JST_B2B, J115 JST_B2B, J116 JST_B4B, J117 JST_B2B, Q101 STN3NF06L, Q102 STN3NF06L, Q103 UNH3N, Q104 NVTA7002NT1G, Q105 RU1E002SPTCL, Q106 NVTA7002NT1G, Q107 NVTA7002NT1G, Q108 RU1E002SPTCL, Q109 NVTA7002NT1G, Q110 RU1E002SPTCL, Q111 DTC143Z, Q112 DTC143Z, Q113 CSD17313Q2, SW102 SW_Push, SW103 SW_Push, U101 XC6220B331MR, U102 nPM1300, U103 ESP32-WROOM-32E, U104 TPS61287, U105 USBLC6-2P6, U106 CP2102N-A02-GQFN24, U107 DS3231M, U108 AT24CS01-SSHM

Commit message: removed gate pull down resistor and re-made erase and boot sequence of ESP32
Parts:
- removed C146: 100nF, Capacitor_SMD:C_0402_1005Metric, symbol Device:C_Small
- removed Q111, Q112: DTC143Z, Package_TO_SOT_SMD:SOT-23-3, symbol Transistor_BJT:DTC143Z
- removed R128, R133, R143: 10K, Resistor_SMD:R_0402_1005Metric, symbol Device:R
- removed R159: 5K1, Resistor_SMD:R_0402_1005Metric, symbol Device:R
- C104, C105: now not fitted
- R123, R139, R148, R149, R150, R163: value 1K -> 10K
- R134, R135, R136, R137, R138, R147: value 0R -> 10K
- R155, R157, R158: value 12K -> 22K
Connections:
- net DTR_SERIAL: no longer R157.1
- net ESP_EN: no longer R158.1
- net GND: now also R155.1, R157.1, R158.1
- net RTS_SERIAL: no longer R155.1
- net VDD: no longer R158.2
- net at J110.1 (Pin_1), Q110.1 (D), R161.2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: now also R158.2
- net at Q110.2 (G), R142.1, TP111.1: now also Q109.2 (D)
- net at Q105.2 (G), R129.1, TP113.1: now also Q106.2 (D)
- net at J105.2 (Pin_2), Q105.1 (D), R162.2: now also R157.2
- net at Q108.1 (D), R160.2, TP137.1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: now also R155.2
- net at Q107.2 (D): now also Q108.2 (G), R132.1, TP126.1
Other:
- note added: "BOOT and RESET"
- note removed: "USB to SERIAL PROGRAMMING"
- moved on the sheet: D111, D112, D113, J105, Q103A, Q103B, R160, R161, R162, TP109, TP131, TP132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

Commit message: Added USB-C PD / Replaced PMIC with TI BMU / Replaced BOOST converter
Parts:
- removed C120: 47uF, Capacitor_SMD:C_0603_1608Metric, symbol Device:C_Small
- removed C121: 47uF, Capacitor_SMD:C_1206_3216Metric, symbol Device:C_Small
- removed C122, C124: 100nF, Capacitor_SMD:C_0402_1005Metric, symbol Device:C_Small
- removed C123: 10uF, Capacitor_SMD:C_0603_1608Metric, symbol Device:C_Small
- removed C125: 58pF, Capacitor_SMD:C_0402_1005Metric, symbol Device:C_Small
- removed C126: 4.7nF, Capacitor_SMD:C_0402_1005Metric, symbol Device:C_Small
- removed C127: 2.2uF, Capacitor_SMD:C_0603_1608Metric, symbol Device:C_Small
- removed C134: 22uF, Capacitor_SMD:C_0603_1608Metric, symbol Device:C_Polarized_Small_US
- removed D108, D109, D110: SS14M, Custom_Global_Footprints:SS14M_Flyback_Diode, symbol Device:D
- removed JP101: ModSel, Jumper:SolderJumper-3_P1.3mm_Open_RoundedPad1.0x1.5mm, symbol Jumper:SolderJumper_3_Open
- removed L103: 4.7uH (SPM12565VT-4R7M-D), Custom_Global_Footprints:SPM12565VT-4R7M, symbol Device:L
- removed Q113: CSD17313Q2, Package_SON:Texas_DQK, symbol Transistor_FET:CSD17313Q2
- removed R116, R118: 5K1, Resistor_SMD:R_0402_1005Metric, symbol Device:R
- removed TP102, TP120, TP121, TP122, TP123, TP125: ~, TestPoint:TestPoint_Pad_D1.0mm, symbol Connector:TestPoint
- removed U102: nPM1300, Package_DFN_QFN:QFN-32-1EP_5x5mm_P0.5mm_EP3.6x3.6mm_ThermalVias, symbol Global_Custom_Libb:nPM1300
- removed U104: TPS61287, Custom_Global_Footprints:RZP0014A-MFG, symbol Global_Custom_Libb:TPS61287
- added C100, C149: 1uF, Capacitor_SMD:C_0603_1608Metric, symbol Device:C
- added C11, C12: 47uF, Capacitor_SMD:CP_Elec_6.3x7.7, symbol Device:C_Polarized_US
- added C134, C156, C157: 100nF, Capacitor_SMD:C_0402_1005Metric, symbol Device:C_Small
- added C146: 100nF, Capacitor_SMD:C_0402_1005Metric, symbol Device:C
- added C150, C151, C153: 10uF, Capacitor_SMD:C_0603_1608Metric, symbol Device:C
- added C152, C154: 10nF, Capacitor_SMD:C_0402_1005Metric, symbol Device:C
- added C155: 10uF, Capacitor_SMD:C_0402_1005Metric, symbol Device:C_Small
- added C158, C160, C161: 1uF, Capacitor_SMD:C_0402_1005Metric, symbol Device:C_Small
- added C159: 3.3uF, Capacitor_SMD:C_0402_1005Metric, symbol Device:C_Small
- added D1, D2, D3, D4: SBR3U40S1F, Diode_SMD:Nexperia_CFP3_SOD-123W, symbol Device:D
- added D115, D116, D117, D118: SML-P12U2TT86R, LED_SMD:LED_0402_1005Metric, symbol Device:LED
- added L2: 10uH, Custom_footprint:SWPA5040S, symbol Device:L
- added L3: 1uH, Custom_footprint:SWPA5040S, symbol Device:L
- added Q111, Q112: DMP6050SSD, Package_SO:SOIC-8_3.9x4.9mm_P1.27mm, symbol Transistor_FET:DMP6050SSD
- added Q113, Q114: DMP3013SFV, Package_SON:Diodes_PowerDI3333-8, symbol Transistor_FET:DMP3013SFV
- added Q115: 2N7002K, Package_TO_SOT_SMD:SOT-23, symbol Transistor_FET:2N7002K
- added Q116: NVTA7002NT1G, Package_TO_SOT_SMD:SOT-323_SC-70, symbol Transistor_FET:RS9N50D
- added Q117: RU1E002SPTCL, Package_TO_SOT_SMD:SOT-323_SC-70, symbol Simulation_SPICE:PMOS
- added R100, R143, R167, R169, R172, R173, R175, R180, R182, R184: 10K, Resistor_SMD:R_0402_1005Metric, symbol Device:R
- added R101: 2M, Resistor_SMD:R_0402_1005Metric, symbol Device:R
- added R128: 121K, Resistor_SMD:R_0402_1005Metric, symbol Device:R
- added R133, R183: 1K, Resistor_SMD:R_0402_1005Metric, symbol Device:R
- added R159, R165: 2K2, Resistor_SMD:R_0402_1005Metric, symbol Device:R
- added R166: 49K9, Resistor_SMD:R_0402_1005Metric, symbol Device:R
- added R168, R170, R171, R174: 0R, Resistor_SMD:R_0402_1005Metric, symbol Device:R
- added R177: 260R, Resistor_SMD:R_0402_1005Metric, symbol Device:R
- added R178: 5K25, Resistor_SMD:R_0402_1005Metric, symbol Device:R
- added R179: 30K1, Resistor_SMD:R_0402_1005Metric, symbol Device:R
- added R181: 22K, Resistor_SMD:R_0402_1005Metric, symbol Device:R
- added R185: 470R, Resistor_SMD:R_0402_1005Metric, symbol Device:R
- added TH101: 103AT-2, symbol Device:Thermistor
- added TP114: ~, TestPoint:TestPoint_Pad_D1.0mm, symbol Connector:TestPoint
- added TP15, TP17, TP25, TP26, TP27: TestPoint_Small, TestPoint:TestPoint_Pad_D1.0mm, symbol Connector:TestPoint_Small
- added U100: TLV61048, Custom_footprint:TLV61048, symbol Custom_Library:TLV61048
- added U104: CYPD3177-24LQ, Package_DFN_QFN:QFN-24-1EP_4x4mm_P0.5mm_EP2.75x2.75mm, symbol Interface_USB:CYPD3177-24LQ
- added U109: NCP1117ST12T3G, Package_TO_SOT_SMD:SOT-223, symbol Regulator_Linear:NCP1117-12_TO252
- added U110: BQ25892, Package_DFN_QFN:WQFN-24-1EP_4x4mm_P0.5mm_EP2.45x2.45mm_ThermalVias, symbol Global_Custom_Libb:BQ25892
- C101: footprint Capacitor_SMD:C_0402_1005Metric -> (none)
- C106: value 1uF -> 10uF; footprint Capacitor_SMD:C_0402_1005Metric -> (none)
- C107, C108: value 10uF -> 47nF; footprint Capacitor_SMD:C_0402_1005Metric -> (none)
- C112: value 2.2uF -> 10uF
- C113: value 100nF -> 47nF; footprint Capacitor_SMD:C_0402_1005Metric -> (none)
- C119: value 100nF -> 4.7uF
- C135: value 4.7nF -> 100nF; now fitted
- R108: value 158K -> 4K7
- R109: value 14K3 -> 4K7
- R110: value 10K -> 4K7
- R111: value 40K -> 220R
- R121: value 10K -> 1K; now fitted
- R139: value 10K -> 1K
Connections:
- net +12V: now also C12.1, C153.1, C154.1, D3.1 (K), D4.1 (K), TP27.1, U109.2 (VO); no longer C119.1, R108.1
- net +3V3: now also R180.2; no longer C113.1
- net +VBAT: now also J117.1 (Pin_1), U110.13 (BAT), U110.14 (BAT); no longer J117.2 (Pin_2)
- net +VSYS: now also C113.1, D115.2 (A), D116.2 (A), D2.2 (A), L3.2, U110.15 (SYS), U110.16 (SYS); no longer C107.1
- net GND: now also J117.2 (Pin_2), C100.2, C11.2, C12.2, C134.2, C146.2, C149.2, C150.2, C151.2, C152.2, C153.2, C154.2, C155.2, C156.2, C157.2, C158.2, C159.2, D118.1 (K), Q115.2 (S), Q116.3 (S), R128.2, R168.2, R170.2, R172.2, R174.2, R175.2, R177.1, R179.1, R181.1, R184.1, TH101.2, U100.2 (GND), U104.19 (GND), U104.22 (GND), U104.25 (GND), U109.1 (GND), U110.17 (PGND), U110.18 (PGND), U110.25 (PGND); no longer C107.2, J103.S1 (SHIELD), J117.1 (Pin_1), R111.1
- net PMIC_SHPHLD: no longer R134.2, U103.8 (IO32)
- net SCL: now also U104.13 (HPI_SCL), U110.5 (SCL)
- net SDA: now also U104.12 (HPI_SDA), U110.6 (SDA)
- net USB_CC1_PD: now also U104.15 (CC1)
- net USB_CC2_PD: now also U104.14 (CC2)
- net VBUS: now also D117.2 (A), Q111.5 (D2), Q111.6 (D2), R166.1, U104.18 (VBUS_IN); no longer C106.1, C128.1, C129.1, R113.1, TP115.1, U106.7 (VREGIN)
- net at C114.2, J112.1 (Pin_1), Q102.2 (D)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: now also D3.2 (A)
- net at R110.1: now also D117.1 (K)
- net at R110.2: now also Q115.3 (D)
- net at R109.1: now also R111.1, U104.9 (FAULT); no longer R108.2
- net at R111.2: now also Q115.1 (G)
- net at Q108.1 (D), R155.2, R160.2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: now also U100.4 (EN)
- net at C133.2, J113.1 (Pin_1), Q101.2 (D)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: now also D4.2 (A)
- net +5V: now reaches C101.1
- net +5V: now also C146.1, C160.1, Q112.7 (D1), Q112.8 (D1), Q114.5 (D), Q117.3 (S), R100.1, R182.2, U100.5 (VIN), U104.11 (VDC_OUT), U110.1 (VBUS)
- net at C135.1: now also J103.S1 (SHIELD), C134.1, R175.1; no longer R121.2
- net SW: no longer names the net of R121.1
- net SW: now also U104.4 (SAFE_PWR_EN)
- net VBUSD renamed +VBUS
- net +VBUS: now also C128.1, C129.1, R113.1, TP115.1, U106.7 (VREGIN), C159.1, C161.1, Q113.5 (D), R143.1
- net VDD renamed +VDD
- new net: R178.1, R179.2, TH101.1, U110.11 (TS)
- new net: C100.1, D2.1 (K), L2.1, TP17.1
- new net: Q116.2 (D), Q117.2 (G), R182.1
- new net: Q116.1 (G), R185.2, TP114.1
- new net: C106.1, U110.23 (PMID)
- new net: D118.2 (A), R183.1
- new net: C107.1, L3.1, U110.19 (SW), U110.20 (SW)
- new net: C160.2, C161.2, Q113.4 (G), Q114.4 (G), R133.2, R143.2
- new net: Q111.4 (G2), Q112.2 (G1), R121.2, R166.2
- new net: Q113.1 (S), Q113.2 (S), Q113.3 (S), Q114.1 (S), Q114.2 (S), Q114.3 (S)
- new net: R101.2, R128.1, TP15.1, U100.3 (FB)
- new net: R100.2, U100.6 (FREQ)
- new net: Q111.3 (S2), Q112.1 (S1)
- new net: D115.1 (K), R159.1
- new net: R159.2, U110.4 (STAT)
- new net: R108.2, U104.10 (FLIP)
- new net: C119.1, R178.2, U110.22 (REGN)
- new net: C158.1, U104.24 (VCCD)
- new net: R177.2, U110.10 (ILIM)
- new net: C107.2, U110.21 (BTST)
- new net: R165.2, U110.3 (~{PG})
- new net: D116.1 (K), R165.1
- new net +14V: C11.1, C149.1, C150.1, C151.1, C152.1, D1.1 (K), R101.1, TP26.1, U109.3 (VI)
- new net +VDDD: C155.1, C156.1, C157.1, R108.1, R167.1, R169.1, R171.1, R173.1, U104.23 (VDDD)
- new net BOOST_IND: D1.2 (A), L2.2, TP25.1, U100.1 (SW)
- new net CE: U110.9 (~{CE})
- new net HPI_INT: U104.7 (~{HPI_INT})
- new net INT: R180.1, U110.7 (INT)
- new net ISNK_COARSE: R171.2, R172.1, U104.5 (ISNK_COARSE)
- new net ISNK_FINE: R173.2, R174.1, U104.6 (ISNK_FINE)
- new net OTG: U110.8 (OTG)
- new net PSEL: Q117.1 (D), R181.2, R183.2, U110.2 (PSEL)
- new net VBUS_FET_EN: R133.1, R184.2, R185.1, U104.3 (VBUS_FET_EN)
- new net VBUS_MAX: R167.2, R168.1, U104.2 (VBUS_MAX)
- new net VBUS_MIN: R169.2, R170.1, U104.1 (VBUS_MIN)
- new net WAKE_SLEEP: R134.2, U103.8 (IO32), U110.12 (~{QON})
- no-connect marks 24 -> 18
Other:
- note added: "+12V LDO for noise filtering"
- note added: "2.65V / +5.5V to +14V Boost Converter"
- note added: "3.5V to 4.35V"
- note added: "Delta IL = usually 30%-40% * IL(DC) Delta IL = 0.4% * 5.83A Delta IL = 2.33A"
- note added: "Host or Adapter PSEL"
- note added: "Inductor Selection IL(DC) = (Vout*Iout)/(Vin*efficiancy) IL(DC) = (14V * 1A) / (3V * 80%) = 5.83A IL(DC) = 5.83A"
- note added: "L= DeltaIL * [(Vin*(Vout+0.8V - Vin)] / [fsw*(Vout + 0.8V)] L= 2.33A * [3V * (14 + 0.8V - 3V)] / [600KHz * (14V + 0.8V)] = 9.296uH L = 9.296uH"
- note added: "Mounting Holes"
- note added: "Output Voltage: R2 should be kept under 150K as per datasheet R1=(Vout/Vref - 1) * R2 R1=(14V/0.8V-1) * 121K = 2M R1 = 2M R2 = 121K Vout = 14V"
- note added: "Parameters: Vin = 3V used as worst case according to datasheet Vout = 14V Vref voltage of 0.8V as per datasheet"
- note added: "Recommended Cout is 10uF with 25V X5R and 1206 package TMK316BLD106KL Taiyo Yuden"
- note added: "SWPA5040S100MT (10uH by SunLord) datasheed recommended"
- note added: "USB-C Power Delivery"
- note removed: "+3V4/+5V to +12V Boost Converter"
- note removed: "IL peak = Idc+(Ipp/2) IL peak = 7.84A+(1.65A/2) = 8.66A Inductor must have a higher saturation current of 9A"
- note removed: "LiPo Voltage Fully Charged 4.2V Discharged 3.3V"
- note removed: "Peak to Peak Inductor Current Ripple Ipp = 1/L*[(1/(Vout-Vin))+(1/Vin)]*fsw OR Ipp = (Vin*D)/(L*fsw) Ipp = (3.4V * 0.73%) / (4.7uH*340KHz) = 1.65A"
- note removed: "Rlim = 400K / A Rlin = 400K / 10A = 40K"
- note removed: "VOUT = 12V VREF = 1V R109 = 14K3 R108 = [(VOUT - VREF) * R109]/VREF R108 = [(12 - 1)* 14300]/1 = 157300 or 158K R108 = 158K"
- note removed: "Vripple_dis = [(VOUT-VIN)*IOUT]/VOUT*fsw*Cout Vripple_dis = [12V-3.4V*2A]/12*320KHz*(47uF*2) = 48mV Vripp_ESR = ILpeak*Rc_esr Vripp_ESR = 8.66A*30mOhms (at 320KHz esr between 10-50mOhms) = 260mV"
- note removed: "n = power convertion efficiency Idc = (VOUT*IOUT)/(VIN*n) Idc = (12V*2A)/(3.4V*90%) = 7.84A"
- moved on the sheet: BT101, C109, C110, C112, C114, C132, C133, C136, C137, C144, C145, C147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

Commit message: Schematic v0.2 done -> check TO DO list
Parts:
- removed J116: JST_B4B, Connector_JST:JST_EH_B4B-EH-A_1x04_P2.50mm_Vertical, symbol Connector_Generic:Conn_01x04
- removed R148, R149, R150: 10K, Resistor_SMD:R_0402_1005Metric, symbol Device:R
- C108, C113: value 47nF -> 10uF
- R134, R135, R136, R137, R138, R147: value 10K -> 1K
- R178: value 5K25 -> 5K23
Connections:
- net +VBUS: now also Q111.5 (D2), Q111.6 (D2), R166.1
- net CE: now also U103.29 (IO5)
- net INT: now also U103.28 (IO17)
- net OTG: now also U103.7 (IO35)
- net VBUS: no longer Q111.5 (D2), Q111.6 (D2), R166.1
- no-connect marks 18 -> 15
Other:
- note added: "+3V3 LDO"
- note added: "TO DO: Find suitable LED's REG / GREEN etc Fix the MOSFET pinout Find suitable capacitors ( correct foot print and voltage rating ) Re-Check schematic for correct values and symbos Re-Check and Re-Do PDN block diagram and check logic Check the BMU thermistor and resustir values Re-evaluate the sleep/wake logic between RTC / ESP32 / BQ25892 QON pin Check footrpints for all components Re-check pino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"
- moved on the sheet: C101, C106, C107, C108, C109, C110, C112, C113, C117, C118, C119, C147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

Commit message: Added extra LDO for PUMP and Water Sensor / Changed Power fet for USB C PD / Implemented Power Distribution Network and Logic / and various stuff
Parts:
- removed Q115: 2N7002K, Package_TO_SOT_SMD:SOT-23, symbol Transistor_FET:2N7002K
- removed R180, R184: 10K, Resistor_SMD:R_0402_1005Metric, symbol Device:R
- removed R185: 470R, Resistor_SMD:R_0402_1005Metric, symbol Device:R
- removed U109: NCP1117ST12T3G, Package_TO_SOT_SMD:SOT-223, symbol Regulator_Linear:NCP1117-12_TO252
- added C120, C121: 10uF, Capacitor_SMD:C_0603_1608Metric, symbol Device:C_Small
- added C13: 47uF, Capacitor_SMD:CP_Elec_6.3x7.7, symbol Device:C_Polarized_US
- added C162, C164: 10uF, Capacitor_SMD:C_0603_1608Metric, symbol Device:C
- added C163, C165: 10nF, Capacitor_SMD:C_0402_1005Metric, symbol Device:C
- added C166, C167: 100nF, Capacitor_SMD:C_0402_1005Metric, symbol Device:C_Small
- added D108: SML-P12U2TT86R, LED_SMD:LED_0402_1005Metric, symbol Device:LED
- added Q118: NVTA7002NT1G, Package_TO_SOT_SMD:SOT-323_SC-70, symbol Transistor_FET:RS9N50D
- added R148, R150, R176, R186, R187: 10K, Resistor_SMD:R_0402_1005Metric, symbol Device:R
- added R149: 470R, Resistor_SMD:R_0402_1005Metric, symbol Device:R
- added TP128: ~, TestPoint:TestPoint_Pad_D1.0mm, symbol Connector:TestPoint
- added TP28, TP29: TestPoint_Small, TestPoint:TestPoint_Pad_D1.0mm, symbol Connector:TestPoint_Small
- added U102: BDJ2FC0WFP, Package_TO_SOT_SMD:TO-252-5_TabPin3, symbol Regulator_Linear:BDJ2FC0WFP
- added U109: NCP1117-12_SOT223, Package_TO_SOT_SMD:SOT-223-3_TabPin2, symbol Regulator_Linear:NCP1117-12_SOT223
- added U111: XC6220B331MR, Package_TO_SOT_SMD:SOT-23-5, symbol Regulator_Linear:XC6220B331MR
- Q113, Q114: value DMP3013SFV -> SI7615DN-T1-GE3
Connections:
- net +14V: now also C162.1, C163.1, TP28.1, U102.1 (EN), U102.2 (VCC), U109.3 (VI)
- net +3V3: now also TP114.1, C121.1, C167.1, R176.2, U111.5 (VOUT); no longer C110.1, C147.1, R123.2, TP103.1, U101.5 (VOUT)
- net +5V: now also D117.2 (A), R186.2
- net +VBUS: now also C132.1, U104.18 (VBUS_IN), U105.5 (VBUS)
- net +VDD: no longer C132.1, U105.5 (VBUS)
- net +VSYS: now also C120.1, C166.1, R150.2, U111.1 (VIN), U111.3 (CE)
- net CE: now also Q116.2 (D), R150.1; no longer U103.29 (IO5)
- net GND: now also C120.2, C121.2, C13.2, C162.2, C163.2, C164.2, C165.2, C166.2, C167.2, D108.1 (K), Q118.3 (S), R148.1, R187.1, U102.3 (GND), U109.1 (GND), U111.2 (GND)
- net VBUS: no longer D117.2 (A), U104.18 (VBUS_IN)
- net VBUS_FET_SAFE_EN: now reaches Q117.2 (G), R182.1
- net VBUS_FET_SAFE_EN: now also Q111.4 (G2), Q112.2 (G1), R121.2, R166.2; no longer Q116.2 (D)
- net at Q116.1 (G): now also R149.2, TP128.1; no longer TP114.1
- net at R111.2: now also Q118.1 (G)
- net at R110.2: now also Q118.2 (D)
- net +12V renamed +12V_PUMP
- net +12V_PUMP: now also C13.1, C164.1, C165.1, TP29.1, U102.4 (VO); no longer C12.1, C153.1, C154.1, Q110.3 (S), R142.2, TP27.1
- net INT: no longer names the net of U110.7 (INT)
- net INT: no longer U103.28 (IO17)
- net OTG: no longer names the net of U103.7 (IO35)
- net OTG: no longer U110.8 (OTG)
- net VBUS_FET_EN: no longer names the net of R133.1, U104.3 (VBUS_FET_EN)
- new net: D108.2 (A), R176.1
- new net: R186.1, R187.2, U110.8 (OTG)
- new net +12V_WATER: C12.1, C153.1, C154.1, Q110.3 (S), R142.2, TP27.1, U109.2 (VO)
- new net +3V3_MCU: C110.1, C147.1, R123.2, TP103.1, U101.5 (VOUT)
- new net CHARGE_ENABLE: R148.2, R149.1, U103.28 (IO17)
- no-connect marks 15 -> 18
Other:
- note added: "+12V LDO"
- note added: "+3V/+5.5V TO +14V BOOST CONVERTER"
- note added: "+3V3 MCU"
- note added: "+3V3 PERIPHERALS"
- note added: "BATTERY MANAGEMENT IC"
- note added: "BOOT & RESET"
- note added: "CHARGE ENABLE"
- note added: "CP2102N USB TO SERIAL CONVERTER"
- note added: "Charge Enable LOW Charge Disable HIGH (default)"
- note added: "HOST OR ADAPTER PSEL"
- note added: "OFF VGS= 5V-5V = 0V Vth= -1V / -2V5"
- note added: "OLED DISPLAY ENABLE"
- note added: "ON VGS= 0V-5V = -5V Vth= -1V / -2V5"
- note added: "OTG LOW disabled (3.5V to 4.35V) HIGH enabled (boost converter to 5V)"
- note added: "Output Voltage: R2 should be kept under 150K as per datasheet R1=(Vout/Vref - 1) * R2 R1=[(14V/0.8V)-1] * 121K = 2M R1 = 2M R2 = 121K Vout = 14V"
- note added: "PROGRAMMING BOOT & RESET"
- note added: "PSEL is controlled by the VBUS_FET_SAFE_EN pin PSEL HIGH = 500mA PSEL LOW = 3.25A When VBUS_FET_SAFE_EN is enabled (Active LOW) will Pull PMOS gate to 0V and PSEL will see a HIGH sig."
- note added: "PUMP 1"
- note added: "PUMP 2"
- note added: "USB <500mA PSEL = HIGH USB >500mA PSEL = LOW NO USB default PSEL = LOW"
- note added: "USB C POWER DELIVERY"
- note added: "USER INTERFACE BUTTONS"
- note added: "WATER SENSOR ENABLE"
- note removed: "+12V LDO for noise filtering"
- note removed: "+3V3 LDO"
- note removed: "2.65V / +5.5V to +14V Boost Converter"
- note removed: "ADD Linear Regulator for Water Sensor to filter noise"
- note removed: "BOOT & Reset"
- note removed: "BOOT and RESET"
- note removed: "CP2102N USB to Serial Converter"
- note removed: "Host or Adapter PSEL"
- note removed: "OLED Display"
- note removed: "Output Voltage: R2 should be kept under 150K as per datasheet R1=(Vout/Vref - 1) * R2 R1=(14V/0.8V-1) * 121K = 2M R1 = 2M R2 = 121K Vout = 14V"
- note removed: "Power Management IC"
- note removed: "Pump 1"
- note removed: "Pump 2"
- note removed: "USB-C Power Delivery"
- note removed: "User Interface Buttons"
- note removed: "Water Sensor"
- moved on the sheet: C100, C101, C106, C107, C108, C109, C11, C110, C112, C113, C119, C12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

Commit message: Fixed MOSFTE footprints and replaced PFET with a more suitable one
Parts:
- removed Q104, Q106, Q107, Q109, Q116, Q118: NVTA7002NT1G, Package_TO_SOT_SMD:SOT-323_SC-70, symbol Transistor_FET:RS9N50D
- removed Q105, Q108, Q110, Q117: RU1E002SPTCL, Package_TO_SOT_SMD:SOT-323_SC-70, symbol Simulation_SPICE:PMOS
- added Q104, Q105, Q106, Q107: BSS314PE, Custom_Global_Footprints:BSS314PE, symbol Transistor_FET:Q_PMOS_GSD
- added Q108, Q109, Q110, Q115, Q116, Q117: NVTA7002NT1G, Custom_Global_Footprints:NVTA7002N, symbol Transistor_FET:Q_NMOS_GSD
Connections:
- net +12V_WATER: now also Q105.2 (S)
- net +3V3: now also Q107.2 (S)
- net +5V: now also Q104.2 (S)
- net +VSYS: now also Q106.2 (S)
- net CE: now also Q117.3 (D)
- net GND: now also Q108.2 (S), Q109.2 (S), Q110.2 (S), Q115.2 (S), Q116.2 (S), Q117.2 (S)
- net PMIC_SHPHLD: now also Q110.3 (D)
- net PSEL: now also Q104.3 (D)
- net VBUS_FET_SAFE_EN: now also Q104.1 (G)
- net at J110.1 (Pin_1), R158.2, R161.2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: now also Q105.3 (D)
- net at R142.1, TP111.1: now also Q105.1 (G), Q108.3 (D)
- net at R129.1, TP113.1: now also Q107.1 (G), Q109.3 (D)
- net at R127.2, TP112.1: now also Q109.1 (G)
- net at R141.2, TP110.1: now also Q108.1 (G)
- net at J105.2 (Pin_2), R157.2, R162.2: now also Q107.3 (D)
- net at R149.2, TP128.1: now also Q117.1 (G)
- net at R131.2, TP127.1: now also Q116.1 (G)
- net at R132.1, TP126.1: now also Q106.1 (G), Q116.3 (D)
- net at R111.2: now also Q115.1 (G)
- net at R155.2, R160.2, TP137.1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: now also Q106.3 (D)
- net at R125.2, TP108.1: now also Q110.1 (G)
- net at R110.2: now also Q115.3 (D)
