File: 01_Hardware/KiCad_v2/Plantomatic2000.kicad_sch (KiCad schematic)
At the start: 272 parts, among them J100 JST_B2B, J101 USB_C_Receptacle_USB2.0_16P, J102 JST_B4B, J103 JST_B4B, J104 JST_B2B, J105 JST_B2B, J106 Conn_02x05_Odd_Even, J107 Conn_02x03_Odd_Even, J108 JST_B2B, J109 JST_B2B, J110 JST_B2B, J111 JST_B2B, J112 JST_B2B, J113 JST_B2B, J114 JST_B2B, Q100 SI7615DN-T1-GE3, Q101 SI7615DN-T1-GE3, Q102 DMP6050SSD, Q103 UNH3N, Q104 NVTA7002NT1G, Q105 BSS314PE, Q106 NVTA7002NT1G, Q107 BSS314PE, Q108 NVTA7002NT1G, Q109 BSS314PE, Q110 BSS314PE, Q111 STN3NF06L, Q112 STN3NF06L, Q113 NVTA7002NT1G, Q114 NVTA7002NT1G, Q115 NVTA7002NT1G, SW100 SW_Push, SW101 SW_Push, U100 XC6220B331MR, U101 XC6220B331MR, U102 BQ25892, U103 USBLC6-2P6, U104 CP2102N-A02-GQFN24, U105 CYPD3177-24LQ, U106 NCP1117-12_SOT223, U107 BDJ2FC0WFP, U108 TLV61048, U109 ESP32-WROOM-32E, U110 AT24CS01-SSHM, U111 DS3231M

Commit message: Replaced BOOST converter, previous one didn't support +2A but rather 200 to 300mA, TO DO: re-do schematic annotation for BOOST, re-do BOM for BOOST
Parts:
- removed BT100: Battery_Cell, Battery:BatteryHolder_MYOUNG_BS-07-A1BJ001_CR2032, symbol Device:Battery_Cell
- removed C100, C128: 4.7uF, Capacitor_SMD:C_0402_1005Metric, symbol Device:C_Small
- removed C101: 100nF, Capacitor_SMD:C_1206_3216Metric, symbol Device:C_Small
- removed C102, C115, C122, C125, C143: 1uF, Capacitor_SMD:C_0603_1608Metric, symbol Device:C_Small
- removed C103, C127, C132, C135, C137, C140, C144, C152, C165: 10uF, Capacitor_SMD:C_0402_1005Metric, symbol Device:C_Small
- removed C104, C123, C124, C139, C153, C156, C160, C164, C175, C176, C177: 100nF, Capacitor_SMD:C_0603_1608Metric, symbol Device:C_Small
- removed C105: 8.2uF, Capacitor_SMD:C_0603_1608Metric, symbol Device:C_Small
- removed C106, C110, C126, C129, C130, C133, C134, C138, C142, C147, C154, C163, C166, C167, C168, C169, C170, C171, C172, C173, C174: 100nF, Capacitor_SMD:C_0402_1005Metric, symbol Device:C_Small
- removed C107, C117, C118: 10uF, Capacitor_SMD:CP_Elec_6.3x5.8, symbol Device:C_Small
- removed C108, C159, C162: 10uF, Capacitor_SMD:C_0603_1608Metric, symbol Device:C_Small
- removed C109, C113: 100nF, Capacitor_SMD:CP_Elec_6.3x5.8, symbol Device:C_Small
- removed C111: 10uF, Capacitor_SMD:C_1206_3216Metric, symbol Device:C_Small
- removed C112, C114: 4.7uF, Capacitor_SMD:CP_Elec_6.3x5.8, symbol Device:C_Small
- removed C116, C131, C151: 1uF, Capacitor_SMD:C_0402_1005Metric, symbol Device:C_Small
- removed C119, C161: 47uF, Capacitor_SMD:C_0402_1005Metric, symbol Device:C_Polarized_Small
- removed C120, C136, C158: 47uF, Capacitor_SMD:C_0603_1608Metric, symbol Device:C_Polarized_Small
- removed C121: 47nF, Capacitor_SMD:C_0603_1608Metric, symbol Device:C_Small
- removed C141, C145: 47uF, Capacitor_SMD:CP_Elec_6.3x5.8, symbol Device:C_Polarized_Small
- removed C146: 22uF, Capacitor_SMD:CP_Elec_10x10, symbol Device:C_Small
- removed C148: 100nF, Capacitor_SMD:CP_Elec_10x10, symbol Device:C_Small
- removed C149: 10uF, Capacitor_SMD:C_0402_1005Metric, symbol Device:C_Polarized_Small
- removed C150: 10uF, Capacitor_SMD:C_1206_3216Metric, symbol Device:C_Polarized_Small
- removed C155: 220uF, Capacitor_SMD:CP_Elec_10x10, symbol Device:C_Polarized_US
- removed C157: 220uF, Capacitor_SMD:C_0603_1608Metric, symbol Device:C_Polarized_US
- removed D100, D101, D103, D104, D110, D111, D116, D117: SML-P12U2TT86R, LED_SMD:LED_0402_1005Metric, symbol Device:LED
- removed D102, D107: SML-P13PTT86R, LED_SMD:LED_0402_1005Metric, symbol Device:LED
- removed D105, D106, D112: SML-P13PTT86R, Custom_Global_Footprints:SBR3U40S1F-7, symbol Device:LED
- removed D108, D109, D113: SBR3U40S1F, Custom_Global_Footprints:SBR3U40S1F-7, symbol Device:D
- removed D114, D115: SBR3U40S1F, LED_SMD:LED_0402_1005Metric, symbol Device:D
- removed H100, H101, H102, H103, H104, H105: MountingHole_Pad, MountingHole:MountingHole_2.2mm_M2_Pad_TopBottom, symbol Mechanical:MountingHole_Pad
- removed J100, J104, J105, J108, J109, J110, J111, J114: JST_B2B, Connector_JST:JST_EH_B2B-EH-A_1x02_P2.50mm_Vertical, symbol Connector_Generic:Conn_01x02
- removed J101: USB_C_Receptacle_USB2.0_16P, Connector_PinHeader_1.27mm:PinHeader_2x05_P1.27mm_Vertical_SMD, symbol Connector:USB_C_Receptacle_USB2.0_16P
- removed J102: JST_B4B, Connector_PinHeader_1.27mm:PinHeader_2x03_P1.27mm_Vertical_SMD, symbol Connector_Generic:Conn_01x04
- removed J103: JST_B4B, Connector_USB:USB_C_Receptacle_Palconn_UTC16-G, symbol Connector_Generic:Conn_01x04
- removed J106: Conn_02x05_Odd_Even, Connector_JST:JST_EH_B2B-EH-A_1x02_P2.50mm_Vertical, symbol Connector_Generic:Conn_02x05_Odd_Even
- removed J107: Conn_02x03_Odd_Even, Connector_JST:JST_EH_B2B-EH-A_1x02_P2.50mm_Vertical, symbol Connector_Generic:Conn_02x03_Odd_Even
- removed J112, J113: JST_B2B, Connector_JST:JST_EH_B4B-EH-A_1x04_P2.50mm_Vertical, symbol Connector_Generic:Conn_01x02
- removed L100: SRN6045HA-1R0Y, Custom_Global_Footprints:SRN6045HA-1R0Y, symbol Device:L
- removed L101: ETQ-P5M100YFM, Custom_Global_Footprints:ETQ-P5M100YFM, symbol Device:L
- removed Q100: SI7615DN-T1-GE3, Custom_Global_Footprints:NVTA7002N, symbol Transistor_FET:DMP3013SFV
- removed Q101: SI7615DN-T1-GE3, Custom_Global_Footprints:BSS314PE, symbol Transistor_FET:DMP3013SFV
- removed Q102: DMP6050SSD, Package_SON:Diodes_PowerDI3333-8, symbol Transistor_FET:DMP6050SSD
- removed Q103: UNH3N, Package_SON:Diodes_PowerDI3333-8, symbol Transistor_BJT:Q_Dual_NPN_NPN_BRT_No_R2_E1B1C2E2B2C1
- removed Q104: NVTA7002NT1G, Custom_Global_Footprints:BSS314PE, symbol Transistor_FET:Q_NMOS_GSD
- removed Q105: BSS314PE, Package_SO:SOIC-8_3.9x4.9mm_P1.27mm, symbol Transistor_FET:Q_PMOS_GSD
- removed Q106, Q113, Q114: NVTA7002NT1G, Custom_Global_Footprints:NVTA7002N, symbol Transistor_FET:Q_NMOS_GSD
- removed Q107, Q109: BSS314PE, Custom_Global_Footprints:NVTA7002N, symbol Transistor_FET:Q_PMOS_GSD
- removed Q108, Q115: NVTA7002NT1G, Package_TO_SOT_SMD:SOT-223, symbol Transistor_FET:Q_NMOS_GSD
- removed Q110: BSS314PE, Custom_Global_Footprints:BSS314PE, symbol Transistor_FET:Q_PMOS_GSD
- removed Q111: STN3NF06L, Custom_Global_Footprints:BSS314PE, symbol Global_Custom_Libb:IRLL014N_HEXFET
- removed Q112: STN3NF06L, Package_TO_SOT_SMD:SOT-363_SC-70-6, symbol Global_Custom_Libb:IRLL014N_HEXFET
- removed R100, R101, R104, R105, R107, R112, R113, R117, R135, R146, R162, R185: 1K, Resistor_SMD:R_0402_1005Metric, symbol Device:R
- removed R102, R111, R114, R123, R124, R125, R126, R128, R129, R132, R136, R138, R140, R141, R147, R149, R150, R152, R165, R166, R171, R172, R174, R175, R176: 10K, Resistor_SMD:R_0402_1005Metric, symbol Device:R
- removed R103, R134, R145, R161, R163: 22K1, Resistor_SMD:R_0402_1005Metric, symbol Device:R
- removed R106, R110, R127, R130, R131, R133, R151, R155, R156, R177, R178, R179, R180, R181, R182, R183, R184: 0R, Resistor_SMD:R_0402_1005Metric, symbol Device:R
- removed R108: 49K9, Resistor_SMD:R_0402_1005Metric, symbol Device:R
- removed R109: 47K5, Resistor_SMD:R_0402_1005Metric, symbol Device:R
- removed R115, R116, R157: 220R, Resistor_SMD:R_0402_1005Metric, symbol Device:R
- removed R118: 5K23, Resistor_SMD:R_0402_1005Metric, symbol Device:R
- removed R119: 130R, Resistor_SMD:R_0402_1005Metric, symbol Device:R
- removed R120, R137, R148, R167, R168, R169, R170, R173: 470R, Resistor_SMD:R_0402_1005Metric, symbol Device:R
- removed R121: 30K1, Resistor_SMD:R_0402_1005Metric, symbol Device:R
- removed R122, R139, R142, R153, R154, R158, R159, R160, R164: 4K7, Resistor_SMD:R_0402_1005Metric, symbol Device:R
- removed R143: 1M, Resistor_SMD:R_0402_1005Metric, symbol Device:R
- removed R144: 64K9, Resistor_SMD:R_0402_1005Metric, symbol Device:R
- removed SW100, SW101: SW_Push, Button_Switch_SMD:SW_SPST_PTS645, symbol Switch:SW_Push
- removed TH100: 103AT-2, symbol Device:Thermistor
- removed TP100, TP101, TP102, TP103, TP105, TP113, TP114, TP115, TP116, TP117, TP118, TP119, TP120, TP121, TP122, TP123, TP124, TP125, TP126, TP127, TP128, TP129, TP130, TP131, TP132, TP133, TP134: ~, TestPoint:TestPoint_Pad_D1.0mm, symbol Connector:TestPoint
- removed TP104: +VBAT, TestPoint:TestPoint_Pad_D1.0mm, symbol Connector:TestPoint
- removed TP106, TP107, TP108, TP109, TP110, TP111, TP112: TestPoint_Small, TestPoint:TestPoint_Pad_D1.0mm, symbol Connector:TestPoint_Small
- removed U100: XC6220B331MR, Package_TO_SOT_SMD:SOT-23-5, symbol Regulator_Linear:XC6220B331MR
- removed U101: XC6220B331MR, Package_DFN_QFN:WQFN-24-1EP_4x4mm_P0.5mm_EP2.45x2.45mm_ThermalVias, symbol Regulator_Linear:XC6220B331MR
- removed U102: BQ25892, RF_Module:ESP32-WROOM-32E, symbol Global_Custom_Libb:BQ25892
- removed U103: USBLC6-2P6, Package_TO_SOT_SMD:SOT-23-5, symbol Global_Custom_Lib:USBLC6-2P6_Custom
- removed U104: CP2102N-A02-GQFN24, Custom_Global_Footprints:TLV61048, symbol Interface_USB:CP2102N-Axx-xQFN24
- removed U105: CYPD3177-24LQ, Package_DFN_QFN:QFN-24-1EP_4x4mm_P0.5mm_EP2.75x2.75mm, symbol Interface_USB:CYPD3177-24LQ
- removed U106: NCP1117-12_SOT223, Package_TO_SOT_SMD:TO-252-5_TabPin3, symbol Regulator_Linear:NCP1117-12_SOT223
- removed U107: BDJ2FC0WFP, Package_TO_SOT_SMD:SOT-666, symbol Regulator_Linear:BDJ2FC0WFP
- removed U108: TLV61048, Package_DFN_QFN:QFN-24-1EP_4x4mm_P0.5mm_EP2.7x2.6mm_ThermalVias, symbol Custom_Library:TLV61048
- removed U109: ESP32-WROOM-32E, Package_TO_SOT_SMD:SOT-223-3_TabPin2, symbol RF_Module:ESP32-WROOM-32E
- removed U110: AT24CS01-SSHM, Package_SO:SOIC-16W_7.5x10.3mm_P1.27mm, symbol Memory_EEPROM:AT24CS01-SSHM
- removed U111: DS3231M, Package_SO:SOIC-8_3.9x4.9mm_P1.27mm, symbol Timer_RTC:DS3231M
Connections:
- no-connect marks 18 -> 0
Other:
- added sheet BATTERY_MANAGEMENT_IC (BATTERY_MANAGEMENT_IC.kicad_sch)
- added sheet CONNECTORS (CONNECTORS.kicad_sch)
- added sheet DC_DC_REGULATORS (DC_DC_REGULATORS.kicad_sch)
- added sheet DISPLAY_AND_WATER_ENABLE (DISPLAY_AND_WATER_ENABLE.kicad_sch)
- added sheet MICROCONTROLLER (MICROCONTROLLER.kicad_sch)
- added sheet PUMPS (PUMPS.kicad_sch)
- added sheet USB_C_POWER_DELIVERY (USB_C_POWER_DELIVERY.kicad_sch)
- added sheet USB_C_TO_SERIAL (USB_C_TO_SERIAL.kicad_sch)
- note removed: "+12V LDO PUMPS"
- note removed: "+12V LDO WATER"
- note removed: "+3V/+5.5V TO +13V BOOST CONVERTER"
- note removed: "+3V3 MCU"
- note removed: "+3V3 PERIPHERALS"
- note removed: "10uH 20% I 5.7A Sat 10.7A DCR 41,3 mohms"
- note removed: "1uH 30% I 6.5A Sat 14.5A DCR 9 mohms"
- note removed: "3.5V to 4.35V"
- note removed: "BATTERY MANAGEMENT IC"
- note removed: "BOOT & RESET"
- note removed: "CHARGE ENABLE"
- note removed: "CP2102N USB TO SERIAL CONVERTER"
- note removed: "Charge Enable LOW Charge Disable HIGH (default)"
- note removed: "Delta IL = usually 30%-40% * IL(DC) Delta IL = 0.4% * 5.83A Delta IL = 2.33A"
- note removed: "EEPROM"
- note removed: "ERA-2AEB3012X"
- note removed: "ERJ-2RKF6492X <- 1%"
- note removed: "ESP32 WROOM 32E"
- note removed: "ESP32: GPIO4 INTERNAL PULL UP TO 3V3 WATER SENSOR: GPIO4 to PIN2 (THE WATER SENSOR SIGNAL)"
- note removed: "HOST OR ADAPTER PSEL"
- note removed: "Hour"
- note removed: "ILIM set to 3A max"
- note removed: "IO12 should be kept low when the module is powered ON"
- note removed: "Inductor Selection IL(DC) = (Vout*Iout)/(Vin*efficiancy) IL(DC) = (14V * 1A) / (3V * 80%) = 5.83A IL(DC) = 5.83A"
- note removed: "JTAG"
- note removed: "L= DeltaIL * [(Vin*(Vout+0.8V - Vin)] / [fsw*(Vout + 0.8V)] L= 2.33A * [3V * (14 + 0.8V - 3V)] / [600KHz * (14V + 0.8V)] = 9.296uH L = 9.296uH"
- note removed: "Line Select"
- note removed: "Manual Start"
- note removed: "Minute"
- note removed: "Mounting Holes"
- note removed: "OFF VGS= 5V-5V = 0V Vth= -1V / -2V5"
- note removed: "OLED DISPLAY ENABLE"
- note removed: "ON VGS= 0V-5V = -5V Vth= -1V / -2V5"
- note removed: "OTG LOW disabled (3.5V to 4.35V) HIGH enabled (boost converter to 5V)"
- note removed: "Output Voltage: R2 should be kept under 150K as per datasheet R1=(Vout/Vref - 1) * R2 R1=[(13V/0.8V)-1] * 64K9 = 1M R1 = 1M R2 = 64K9K Vout = 13V"
- note removed: "PROGRAMMING BOOT & RESET"
- note removed: "PSEL is controlled by the VBUS_FET_SAFE_EN pin PSEL HIGH = 500mA PSEL LOW = 3.25A When VBUS_FET_SAFE_EN is enabled (Active LOW) will Pull PMOS gate to 0V and PSEL will see a HIGH sig."
- note removed: "PUMP 1"
- note removed: "PUMP 2"
- note removed: "Parameters: Vin = 3V used as worst case according to datasheet Vout = 14V Vref voltage of 0.8V as per datasheet"
- note removed: "RC delay circuit"
- note removed: "RE0402BRE071ML"
- note removed: "RG1005P-131-B-T5"
- note removed: "RGC1/16SC6492BTH"
- note removed: "RT0402BRE075K23L"
- note removed: "RTC DS3231"
- note removed: "Recommended Cout is 10uF with 25V X5R and 1206 package TMK316BLD106KL Taiyo Yuden"
- note removed: "Running LED"
- note removed: "System Reset"
- note removed: "System WakeUp"
- note removed: "UART_PROG"
- note removed: "USB <500mA PSEL = HIGH USB >500mA PSEL = LOW NO USB default PSEL = LOW"
- note removed: "USB C POWER DELIVERY"
- note removed: "USER INTERFACE BUTTONS"
- note removed: "UUX1E221MNL1GS"
- note removed: "UWT1V470MCL1GS"
- note removed: "VBUS is used to sense if USB is connected VBUS must not exceed VIO (which is VDD -> which is 3V3 from the internal LDO) +2.5V Voltage divider (5V * 47K5) / (22K1 + 47K5) = 3.4V"
- note removed: "VDD is supplied by the VDD pin of CP2102N When USB C is removed the CP2102N should power OFF"
- note removed: "WATER SENSOR ENABLE"

Commit message: Hardware for manufacturing v0.2
Other:
- sheet MICROCONTROLLER ports: added ESP_RX, ESP_TX; removed none
- sheet USB_C_TO_SERIAL ports: added ESP_RX, ESP_TX; removed none
Changed lines of the file:
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@@
+	(wire
+		(pts
+			(xy 165.1 101.6) (xy 165.1 139.7)
+		)
+		(stroke
+			(width 0)
+			(type default)
+		)
+	)
 	(wire
 		(pts
@@
 	(wire
 		(pts
-			(xy 167.64 106.68) (xy 167.64 127)
+			(xy 170.18 93.98) (xy 170.18 127)
 		)
 		(stroke
@@
 	(wire
 		(pts
-			(xy 158.75 106.68) (xy 167.64 106.68)
+			(xy 158.75 139.7) (xy 165.1 139.7)
+		)
+		(stroke
+			(width 0)
+			(type default)
+		)
+	)
+	(wire
+		(pts
+			(xy 158.75 93.98) (xy 170.18 93.98)
 		)
 		(stroke
@@
 	(wire
 		(pts
-			(xy 167.64 127) (xy 175.26 127)
+			(xy 170.18 127) (xy 175.26 127)
 		)
 		(stroke
@@
 	(wire
 		(pts
+			(xy 167.64 97.79) (xy 158.75 97.79)
+		)
+		(stroke
+			(width 0)
+			(type default)
+		)
+	)
+	(wire
+		(pts
 			(xy 158.75 81.28) (xy 175.26 81.28)
 		)
@@
 	(wire
 		(pts
+			(xy 167.64 143.51) (xy 167.64 97.79)
+		)
+		(stroke
+			(width 0)
+			(type default)
+		)
+	)
+	(wire
+		(pts
+			(xy 158.75 143.51) (xy 167.64 143.51)
+		)
+		(stroke
+			(width 0)
+			(type default)
+		)
+	)
+	(wire
+		(pts
 			(xy 109.22 115.57) (xy 109.22 101.6)
+		)
+		(stroke
+			(width 0)
+			(type default)
+		)
+	)
+	(wire
+		(pts
+			(xy 158.75 101.6) (xy 165.1 101.6)
 		)
 		(stroke
@@
 			)
 		)
+		(pin "ESP_TX" input
+			(at 158.75 143.51 0)
+			(effects
+				(font
+					(size 1.27 1.27)
+				)
+				(justify right)
+			)
+		)
+		(pin "ESP_RX" output
+			(at 158.75 139.7 0)
+			(effects
+				(font
+					(size 1.27 1.27)
+				)
+				(justify right)
+			)
+		)
 		(instances
 			(project "Plantomatic2000"
@@
 		)
 		(pin "BOOST_ENABLE" output
-			(at 158.75 106.68 0)
+			(at 158.75 93.98 0)
 			(effects
 				(font
@@
 			(effects
 				(font
+					(size 1.27 1.27)
+				)
+				(justify right)
+			)
+		)
+		(pin "ESP_TX" output
+			(at 158.75 97.79 0)
+			(effects
+				(font
+					(size 1.27 1.27)
+				)
+				(justify right)
+			)
+		)
+		(pin "ESP_RX" input
+			(at 158.75 101.6 0)
+			(effects
+				(font
