File: 01_Hardware/KiCad_v2/DC_DC_REGULATORS.kicad_sch (KiCad schematic)
At the start: 75 parts, among them Q113 CSD17313Q2, Q401 SI7615DN-T1-GE3, Q402 NVTA7002NT1G, U104 TPS61287, U400 BDJ2FC0WFP, U402 NCP1117-12_SOT223, U403 XC6220B331MR, U404 XC6220B331MR

Commit message: BOM done, except connectors/thermistor/button -> Will re-check BOM before sending to manufacturing
Parts:
- removed C119: 100nF, Capacitor_SMD:C_0402_1005Metric, symbol Device:C_Small
- removed C120: 47uF, Capacitor_SMD:C_0603_1608Metric, symbol Device:C_Small
- removed C121: 47uF, Capacitor_SMD:C_1206_3216Metric, symbol Device:C_Small
- removed C134: 22uF, Capacitor_SMD:C_0603_1608Metric, symbol Device:C_Polarized_Small_US
- removed C404, C411, C416: 47uF, Capacitor_SMD:CP_Elec_6.3x5.8, symbol Device:C_Polarized_Small
- removed C405, C407: 1uF, Capacitor_SMD:C_0603_1608Metric, symbol Device:C_Small
- removed D402: NCD0402G1, Custom_Global_Footprints:SML-P13PTT_LED_0402_1005Metric, symbol Device:LED
- removed JP101: ModSel, Jumper:SolderJumper-3_P1.3mm_Open_RoundedPad1.0x1.5mm, symbol Jumper:SolderJumper_3_Open
- removed Q401: SI7615DN-T1-GE3, Package_SON:Diodes_PowerDI3333-8, symbol Transistor_FET:DMP3013SFV
- removed Q402: NVTA7002NT1G, Custom_Global_Footprints:NVTA7002N, symbol Transistor_FET:Q_NMOS_GSD
- removed R401, R402, R407: 10K, Resistor_SMD:R_0402_1005Metric, symbol Device:R
- removed R408: 22K1, Resistor_SMD:R_0402_1005Metric, symbol Device:R
- removed R409: 1K, Resistor_SMD:R_0402_1005Metric, symbol Device:R
- removed TP121, TP122, TP123, TP125, TP404, TP406, TP407, TP410, TP411: ~, TestPoint:TestPoint_Pad_D1.0mm, symbol Connector:TestPoint
- removed TP400, TP401, TP408, TP409: TestPoint_Small, TestPoint:TestPoint_Pad_D1.0mm, symbol Connector:TestPoint_Small
- removed U400: BDJ2FC0WFP, Package_TO_SOT_SMD:TO-252-4, symbol Regulator_Linear:BDJ2FC0WFP
- removed U402: NCP1117-12_SOT223, Package_TO_SOT_SMD:SOT-223, symbol Regulator_Linear:NCP1117-12_SOT223
- added C130, C131: 47uF, Capacitor_SMD:C_1206_3216Metric, symbol Device:C_Small
- added C207, C208: 1uF, Capacitor_SMD:C_0603_1608Metric, symbol Device:C_Small
- added C404, C405: 330uF, Capacitor_Tantalum_SMD:CP_EIA-7343-31_Kemet-D, symbol Device:C_Polarized
- added C406: 470uF, Capacitor_Tantalum_SMD:CP_EIA-7360-38_Kemet-E, symbol Device:C_Polarized
- added C510, C511, C512, C513: 22uF, Capacitor_SMD:C_0805_2012Metric, symbol Device:C_Small
- added D201: NCD0402R1, LED_SMD:LED_0402_1005Metric, symbol Device:LED
- added Q204: SI7615DN-T1-GE3, Package_SON:Diodes_PowerDI3333-8, symbol Transistor_FET:DMP3013SFV
- added Q205: IRLML2402TRPBF, Package_TO_SOT_SMD:SOT-23, symbol Transistor_FET:Q_NMOS_GSD
- added R112: 22K1, Resistor_SMD:R_0402_1005Metric, symbol Device:R
- added R217: 49K9, Resistor_SMD:R_0402_1005Metric, symbol Device:R
- added R218: 1K, Resistor_SMD:R_0402_1005Metric, symbol Device:R
- added TP424, TP425, TP426, TP427, TP428, TP429: TestPoint_Small, TestPoint:TestPoint_Pad_D1.5mm, symbol Connector:TestPoint_Small
- added U405, U406: LM1085IS-12/NOPB, Package_TO_SOT_SMD:TO-263-3_TabPin2, symbol Regulator_Linear:NCP1117-12_SOT223
- C122, C124: Link (none) -> https://jlcpcb.com/partdetail/166764-CL05B104KA5NNNC/C155422; Manufacturer (none) -> Samsung Electro-Mechanics; Manufacturer Part Number (none) -> CL05B104KA5NNNC
- C123: Link (none) -> https://jlcpcb.com/partdetail/320824-GRM188R61E106KA73D/C34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; Manufacturer (none) -> Murata Electronics; Manufacturer Part Number (none) -> GRM188R61E106KA73D
- C125: value 58pF -> 100pF; Link (none) -> https://jlcpcb.com/partdetail/YAGEO-CC0402FRNPO9BN101/C3271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; Manufacturer (none) -> YAGEO; Manufacturer Part Number (none) -> CC0402FRNPO9BN101
- C126: value 4.7nF -> 22nF; Link (none) -> https://jlcpcb.com/partdetail/542588-GCM155R71H223JA55D/C52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; Manufacturer (none) -> Murata Electronics; Manufacturer Part Number (none) -> GCM155R71H223JA55D
- C127: value 2.2uF -> 4.7uF
- C135: value 4.7nF -> 22nF; Manufacturer (none) -> Murata Electronics; Manufacturer Part Number (none) -> GCM155R71H223JA55D
- C400, C403, C412, C415, C417, C420, C421, C424: Manufacturer Murata Electronics -> Murata Electronics
- C401, C402, C413, C414, C418, C419, C422, C423: Manufacturer Samsung Electro-Mechanics -> Samsung Electro-Mechanics
- D400, D403, D404, D405: footprint Custom_Global_Footprints:SML-P13PTT_LED_0402_1005Metric -> LED_SMD:LED_0402_1005Metric
- Q113: Link (none) -> https://jlcpcb.com/partdetail/TexasInstruments-CSD17313Q2/C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; Manufacturer (none) -> Texas Instruments; Manufacturer Part Number (none) -> CSD17313Q2
- R108: Manufacturer (none) -> YAGEO; Manufacturer Part Number (none) -> RC0402FR-07158KL
- R109: Manufacturer (none) -> YAGEO; Manufacturer Part Number (none) -> AC0402FR-0714K3L
- R110: value 10K -> 49K9; Manufacturer (none) -> YAGEO; Manufacturer Part Number (none) -> RC0402FR-0749K9L
- R111: value 40K -> 20K; Manufacturer (none) -> YAGEO; Manufacturer Part Number (none) -> RC0402FR-0720KL
- R121: Manufacturer (none) -> YAGEO; Manufacturer Part Number (none) -> RC0402FR-0710KL
- R400, R410: Manufacturer (none) -> YAGEO; Manufacturer Part Number (none) -> RC0402FR-074K7L
- R405: Manufacturer (none) -> YAGEO; Manufacturer Part Number (none) -> RC0402FR-07470RL
- R411, R412: Manufacturer (none) -> YAGEO; Manufacturer Part Number (none) -> RC0402FR-071KL
- U104: value TPS61287 -> TPS61287RZPR; Manufacturer (none) -> Texas Instruments; Manufacturer Part Number (none) -> TPS61287RZPR
- U403, U404: value XC6220B331MR -> XC6220B331MR-G; Link (none) -> https://jlcpcb.com/partdetail/TorexSemicon-XC6220B331MRG/C8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; Manufacturer (none) -> Torex Semicon; Manufacturer Part Number (none) -> XC6220B331MR-G
Connections:
- net CVCC is gone; now on an unnamed net: C127.1, U104.11 (VCC)
- net +12V: now also C405.1, C406.1, C510.1, C511.1, C512.1, C513.1, TP424.1
- net +12V_PUMP: now also C130.1, TP426.1, U405.2 (VO)
- net +12V_WATER: now also C131.1, TP427.1, U406.2 (VO)
- net +13V: now also U405.3 (VI), U406.3 (VI)
- net +3V3: now also TP429.1
- net +3V3_MCU: now also TP428.1
- net +VSYS: now also C207.1, Q204.1 (S), Q204.2 (S), Q204.3 (S), R217.1; no longer C123.1, C124.1, L103.2, U104.12 (VIN)
- net BOOST_ENABLE: now also R112.1
- net GND: now also C130.2, C131.2, C404.2, C405.2, C406.2, C510.2, C511.2, C512.2, C513.2, Q205.2 (S), R112.2, U405.1 (GND), U406.1 (GND)
- net at U104.13 (EN/UVLO): now also C123.1, C124.1, L103.2, U104.12 (VIN), C208.1, C404.1, Q204.5 (D), R218.1
- net at Q113.3 (G), U104.9 (DRV): now also TP425.1
- net at R405.2: now also Q205.1 (G)
- new net: C207.2, C208.2, D201.1 (K), Q204.4 (G), Q205.3 (D), R217.2
- new net: D201.2 (A), R218.2
Other:
- note removed: "Rlim = 400K / A Rlin = 400K / 10A = 40K"
- moved on the sheet: C122, C123, C124, C125, C126, C127, C135, C400, C401, C402, C403, C412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

Commit message: USB-C and Serial PCB routing done
Other:
- moved on the sheet: C122, C123, C124, C125, C126, C127, C130, C131, C135, C207, C208, C400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

Commit message: Power plane/rearranged connectors
Connections:
- net +13V is gone; now on net +12V: C400.1, C401.1, C412.1, C413.1, U405.3 (VI), U406.3 (VI)
- net BOOST_COMP: now reaches C125.1, R110.1, U104.3 (COMP)
- net B_VCC: now reaches C127.1, U104.11 (VCC), U104.4 (MODE)
- net BOOST_VIN: now reaches C123.1, C124.1, C208.1, C404.1, L103.2, Q204.5 (D), R218.1, U104.12 (VIN), U104.13 (EN/UVLO)
- net BOOST_FB: now reaches R108.2, R109.1, U104.2 (FB)
- net BOOST_ILIM: now reaches R111.2, U104.1 (ILIM)
- net BOOT: now reaches C122.2, U104.7 (BOOT)
- net BOOST_DRV: now reaches Q113.3 (G), TP425.1, U104.9 (DRV)
- net SW renamed BOOT_SW
Other:
- moved on the sheet: C122, C127, L103, R111

Commit message: Hardware for manufacturing v0.2
Parts:
- removed TP425: TestPoint_Small, TestPoint:TestPoint_Pad_D1.5mm, symbol Connector:TestPoint_Small
- TP424, TP426, TP427, TP428, TP429: footprint TestPoint:TestPoint_Pad_D1.5mm -> TestPoint:TestPoint_Pad_D1.0mm
Other:
- moved on the sheet: R109
Changed lines of the file:
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@@
 	)
 	(junction
-		(at 177.8 90.17)
-		(diameter 0)
-		(color 0 0 0 0)
-	)
-	(junction
 		(at 274.32 67.31)
 		(diameter 0)
@@
 	(wire
 		(pts
-			(xy 265.43 77.47) (xy 265.43 78.74)
+			(xy 265.43 77.47) (xy 265.43 82.55)
 		)
 		(stroke
@@
 	(wire
 		(pts
-			(xy 177.8 90.17) (xy 185.42 90.17)
+			(xy 168.91 90.17) (xy 185.42 90.17)
 		)
 		(stroke
@@
 	(wire
 		(pts
-			(xy 168.91 90.17) (xy 177.8 90.17)
-		)
-		(stroke
-			(width 0)
-			(type default)
-		)
-	)
-	(wire
-		(pts
 			(xy 115.57 77.47) (xy 119.38 77.47)
 		)
@@
 	(wire
 		(pts
-			(xy 265.43 86.36) (xy 265.43 88.9)
+			(xy 265.43 90.17) (xy 265.43 92.71)
 		)
 		(stroke
@@
 	(wire
 		(pts
-			(xy 177.8 90.17) (xy 177.8 91.44)
-		)
-		(stroke
-			(width 0)
-			(type default)
-		)
-	)
-	(wire
-		(pts
 			(xy 288.29 95.25) (xy 288.29 99.06)
 		)
@@
 		)
 		(property "Description" "1% 1/16W"
-			(at 238.76 87.63 0)
+			(at 241.046 87.63 90)
 			(effects
 				(font
 					(size 1.27 1.27)
 				)
-				(hide yes)
 			)
 		)
@@
 			)
 		)
-		(property "Datasheet" "~"
+		(property "Datasheet" ""
 			(at 220.98 100.33 0)
 			(effects
@@
 			)
 		)
-		(property "Description" "Unpolarized capacitor, small symbol"
-			(at 220.98 100.33 0)
+		(property "Description" "25V 10%"
+			(at 225.552 102.616 0)
 			(effects
 				(font
 					(size 1.27 1.27)
 				)
-				(hide yes)
 			)
 		)
@@
 		)
 		(property "Description" "1% 1/16W"
-			(at 265.43 72.39 0)
+			(at 267.97 72.898 90)
 			(effects
 				(font
 					(size 1.27 1.27)
 				)
-				(hide yes)
 			)
 		)
@@
 					(size 1.27 1.27)
 				)
-				(hide yes)
 			)
 		)
@@
 	(symbol
 		(lib_id "Device:R")
-		(at 265.43 82.55 0)
+		(at 265.43 86.36 0)
 		(unit 1)
 		(exclude_from_sim no)
@@
 		(dnp no)
 		(property "Reference" "R109"
-			(at 265.43 85.09 90)
+			(at 265.43 88.9 90)
 			(effects
 				(font
@@
 		)
 		(property "Value" "14K3"
-			(at 263.398 85.344 90)
+			(at 263.398 89.154 90)
 			(effects
 				(font
@@
 		)
 		(property "Footprint" "Resistor_SMD:R_0402_1005Metric"
-			(at 263.652 82.55 90)
+			(at 263.652 86.36 90)
 			(effects
 				(font
@@
 		)
 		(property "Datasheet" ""
-			(at 265.43 82.55 0)
+			(at 265.43 86.36 0)
 			(effects
 				(font
@@
 			)
 		)
-		(property "Description" "Resistor"
-			(at 265.43 82.55 0)
+		(property "Description" "1% 1/16W"
+			(at 267.462 86.36 90)
 			(effects
 				(font
 					(size 1.27 1.27)
 				)
-				(hide yes)
 			)
 		)
 		(property "Manufacturer" "YAGEO"
-			(at 265.43 82.55 0)
+			(at 265.43 86.36 0)
 			(effects
 				(font
@@
 		)
 		(property "Manufacturer Part Number" "AC0402FR-0714K3L"
-			(at 265.43 82.55 0)
+			(at 265.43 86.36 0)
 			(effects
 				(font
@@
 					(size 1.27 1.27)
 				)
-				(hide yes)
 			)
 		)
@@
 			)
 		)
-		(property "Footprint" "TestPoint:TestPoint_Pad_D1.5mm"
+		(property "Footprint" "TestPoint:TestPoint_Pad_D1.0mm"
 			(at 261.62 194.31 0)
 			(effects
@@
 		)
 		(property "Description" "1% 1/16W"
-			(at 148.59 87.63 0)
+			(at 150.876 87.63 90)
 			(effects
 				(font
 					(size 1.27 1.27)
 				)
-				(hide yes)
 			)
 		)
@@
 	(symbol
 		(lib_id "power:GNDA")
-		(at 265.43 88.9 0)
+		(at 265.43 92.71 0)
 		(unit 1)
 		(exclude_from_sim no)
@@
 		(dnp no)
 		(property "Reference" "#PWR0143"
-			(at 265.43 95.25 0)
+			(at 265.43 99.06 0)
 			(effects
 				(font
@@
 		)
 		(property "Value" "GNDA"
-			(at 265.43 92.71 0)
+			(at 265.43 96.52 0)
 			(effects
 				(font
@@
 		)
 		(property "Footprint" ""
-			(at 265.43 88.9 0)
+			(at 265.43 92.71 0)
 			(effects
 				(font
@@
 		)
 		(property "Datasheet" ""
-			(at 265.43 88.9 0)
+			(at 265.43 92.71 0)
 			(effects
 				(font
@@
 		)
 		(property "Description" "Power symbol creates a global label with name \"GNDA\" , analog ground"
-			(at 265.43 88.9 0)
+			(at 265.43 92.71 0)
 			(effects
 				(font
@@
 	)
 	(symbol
-		(lib_id "Connector:TestPoint_Small")
-		(at 177.8 91.44 0)
-		(unit 1)
-		(exclude_from_sim no)
-		(in_bom no)
-		(on_board yes)
-		(dnp no)
-		(property "Reference" "TP425"
-			(at 174.752 93.218 0)
-			(effects
-				(font
-					(size 1.27 1.27)
-				)
-				(justify left)
-			)
-		)
-		(property "Value" "TestPoint_Small"
-			(at 179.07 92.7099 0)
-			(effects
-				(font
-					(size 1.27 1.27)
-				)
-				(justify left)
-				(hide yes)
-			)
-		)
-		(property "Footprint" "TestPoint:TestPoint_Pad_D1.5mm"
-			(at 182.88 91.44 0)
-			(effects
-				(font
-					(size 1.27 1.27)
-				)
-				(hide yes)
-			)
-		)
-		(property "Datasheet" ""
-			(at 182.88 91.44 0)
-			(effects
-				(font
-					(size 1.27 1.27)
-				)
-				(hide yes)
-			)
-		)
-		(property "Description" "test point"
-			(at 177.8 91.44 0)
-			(effects
-				(font
-					(size 1.27 1.27)
-				)
-				(hide yes)
-			)
-		)
-		(pin "1"
-		)
-		(instances
-			(project "Plantomatic2000"
-				(path "/7b3f5236-3811-4a22-865a-1f6a26bdd727/9c3e402b-37be-4fff-9c3c-af2f37c1deef"
-					(reference "TP425")
-					(unit 1)
-				)
-			)
-		)
-	)
-	(symbol
 		(lib_id "power:GND")
 		(at 86.36 158.75 0)
@@
 					(size 1.27 1.27)
 				)
-				(hide yes)
 			)
 		)
@@
 			)
 		)
-		(property "Footprint" "TestPoint:TestPoint_Pad_D1.5mm"
+		(property "Footprint" "TestPoint:TestPoint_Pad_D1.0mm"
 			(at 149.86 146.05 0)
 			(effects
@@
 					(size 1.27 1.27)
 				)
-				(hide yes)
 			)
 		)
@@
 					(size 1.27 1.27)
 				)
-				(hide yes)
 			)
 		)
@@
 		)
 		(property "Description" "1% 1/16W"
-			(at 229.87 93.98 0)
+			(at 231.902 93.472 90)
 			(effects
 				(font
 					(size 1.27 1.27)
 				)
-				(hide yes)
 			)
 		)
@@
 			)
 		)
-		(property "Footprint" "TestPoint:TestPoint_Pad_D1.5mm"
+		(property "Footprint" "TestPoint:TestPoint_Pad_D1.0mm"
 			(at 219.71 64.77 0)
 			(effects
@@
 					(size 1.27 1.27)
 				)
-				(hide yes)
 			)
 		)
@@
 			)
 		)
-		(property "Footprint" "TestPoint:TestPoint_Pad_D1.5mm"
+		(property "Footprint" "TestPoint:TestPoint_Pad_D1.0mm"
 			(at 266.7 148.59 0)
 			(effects
@@
 			)
 		)
-		(property "Footprint" "TestPoint:TestPoint_Pad_D1.5mm"
+		(property "Footprint" "TestPoint:TestPoint_Pad_D1.0mm"
 			(at 149.86 195.58 0)
 			(effects
