File: 01_Hardware/KiCad_v2/USB_C_TO_SERIAL.kicad_sch (KiCad schematic)
At the start: 25 parts, among them J100 TYPE-C-31-M-12, Q100 UMH3N, U100 USBLC6-2P6, U101 CP2102N-A02-GQFN24

Commit message: BOM done, except connectors/thermistor/button -> Will re-check BOM before sending to manufacturing
Parts:
- removed TP100, TP101, TP504, TP505: ~, TestPoint:TestPoint_Pad_D1.0mm, symbol Connector:TestPoint
- added TP402, TP403, TP405, TP412: TestPoint_Small, TestPoint:TestPoint_Pad_D1.5mm, symbol Connector:TestPoint_Small
- C101, C102, C104, C105, C106: Manufacturer Samsung Electro-Mechanics -> Samsung Electro-Mechanics
- D100, D101: footprint Custom_Global_Footprints:SML-P13PTT_LED_0402_1005Metric -> LED_SMD:LED_0402_1005Metric
- R100: Manufacturer (none) -> YAGEO; Manufacturer Part Number (none) -> RT0402BRD0722K1L
- R101: Manufacturer (none) -> YAGEO; Manufacturer Part Number (none) -> RC0402FR-071KL
- R102, R104: Manufacturer (none) -> YAGEO; Manufacturer Part Number (none) -> AC0402FR-070RL
- R103: Manufacturer (none) -> YAGEO; Manufacturer Part Number (none) -> AC0402FR-0747K5L
- R105, R106: Manufacturer (none) -> YAGEO; Manufacturer Part Number (none) -> RC0402FR-07220RL
- R107: Manufacturer (none) -> YAGEO; Manufacturer Part Number (none) -> RC0402FR-0710KL
- U100: Manufacturer (none) -> STMicroelectronics; Manufacturer Part Number (none) -> USBLC6-2P6
- U101: value CP2102N-A02-GQFN24 -> CP2102N-A02-GQFN24R; Link (none) -> https://jlcpcb.com/partdetail/1058352-CP2102N_A02GQFN24R/C9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; Manufacturer (none) -> SKYWORKS/SILICON LABS; Manufacturer Part Number (none) -> CP2102N-A02-GQFN24R
Connections:
- net +VBUS: now also TP403.1
- net +VDD: now also TP402.1
- net DTR_SERIAL: now also TP405.1
- net RTS_SERIAL: now also TP412.1
Other:
- moved on the sheet: R100, R103

Commit message: USB-C and Serial PCB routing done
Changed lines of the file:
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@@
 					(size 1.27 1.27)
 				)
+				(hide yes)
 			)
 		)
@@
 					(size 1.27 1.27)
 				)
+				(hide yes)
 			)
 		)
@@
 					(size 1.27 1.27)
 				)
+				(hide yes)
 			)
 		)
@@
 					(size 1.27 1.27)
 				)
+				(hide yes)
 			)
 		)
@@
 					(size 1.27 1.27)
 				)
+				(hide yes)
 			)
 		)
@@
 					(size 1.27 1.27)
 				)
+				(hide yes)
 			)
 		)
@@
 					(size 1.27 1.27)
 				)
+				(hide yes)
 			)
 		)
@@
 					(size 1.27 1.27)
 				)
+				(hide yes)
 			)
 		)
@@
 					(size 1.27 1.27)
 				)
+				(hide yes)
 			)
 		)
@@
 					(size 1.27 1.27)
 				)
+				(hide yes)
 			)
 		)
@@
 					(size 1.27 1.27)
 				)
+				(hide yes)
 			)
 		)
@@
 					(size 1.27 1.27)
 				)
+				(hide yes)
 			)
 		)
@@
 					(size 1.27 1.27)
 				)
+				(hide yes)
 			)
 		)
@@
 					(size 1.27 1.27)
 				)
+				(hide yes)
 			)
 		)
@@
 					(size 1.27 1.27)
 				)
+				(hide yes)
 			)
 		)
@@
 					(size 1.27 1.27)
 				)
+				(hide yes)
 			)
 		)
@@
 					(size 1.27 1.27)
 				)
+				(hide yes)
 			)
 		)
@@
 					(size 1.27 1.27)
 				)
+				(hide yes)
 			)
 		)
@@
 					(size 1.27 1.27)
 				)
+				(hide yes)
 			)
 		)
@@
 					(size 1.27 1.27)
 				)
+				(hide yes)
 			)
 		)
@@
 					(size 1.27 1.27)
 				)
+				(hide yes)
 			)
 		)
@@
 					(size 1.27 1.27)
 				)
+				(hide yes)
 			)
 		)
@@
 					(size 1.27 1.27)
 				)
+				(hide yes)
 			)
 		)
@@
 					(size 1.27 1.27)
 				)
-			)
-		)
+				(hide yes)
+			)
+		)

Commit message: Hardware for manufacturing v0.2
Parts:
- added C407, C408, C409, C410, C411, C416, C425, C426, C427, C428: 4.7nF, Capacitor_SMD:C_0402_1005Metric, symbol Device:C_Small
- added R401, R407, R408, R409, R413, R414, R415, R416, R417, R418: 22R, Resistor_SMD:R_0402_1005Metric, symbol Device:R
- added R402, R403, R404, R406, R419, R420: 511K, Resistor_SMD:R_0402_1005Metric, symbol Device:R
- C100, C103: Manufacturer Samsung Electro-Mechanics -> (none); Manufacturer Part Number CL10A475KA8NQNC -> (none)
- TP402, TP403, TP405, TP412: footprint TestPoint:TestPoint_Pad_D1.5mm -> TestPoint:TestPoint_Pad_D1.0mm
Connections:
- net GND: now also C407.2, C408.2, C409.2, C410.2, C411.2, C416.2, C425.2, C426.2, C427.2, C428.2, R402.1, R403.1, R404.1, R406.1, R419.1, R420.1
- net shield: now reaches C105.1, C106.1, J100.S1 (SHIELD), R107.1
- net shield: now also R401.2, R402.2, R403.2, R404.2, R406.2, R407.2, R408.2, R409.2, R413.2, R414.2, R415.2, R416.2, R417.2, R418.2, R419.2, R420.2
- new net: C410.1, R409.1
- new net: C411.1, R413.1
- new net: C427.1, R417.1
- new net: C416.1, R414.1
- new net: C407.1, R401.1
- new net: C426.1, R416.1
- new net: C409.1, R408.1
- new net: C428.1, R418.1
- new net: C425.1, R415.1
- new net: C408.1, R407.1
Other:
- moved on the sheet: C104
